File: redphone.brd (EAGLE design)
At the start: 139 x 65 mm, 247 parts, among them IC1 EP4CE15E22, IC10 74LVC1G02DCK, IC11 74LVC1G02DCK, IC12 74LVC1G02DCK, IC13 MAX1708, IC15 LSM303DLHC, IC16 EPCS4SI8N, IC17 L3GD20, IC18 WM8903, IC19 AT25SF041, IC2 STM32F429ZIT, IC20 MP34DT01, IC21 PT4181, IC22 MAX8903A, IC23 NRF24L01+, IC24 BME280, IC25 APDS-9960, IC3 MT48LC16M16A2TG, IC4 MAX8815A, IC5 TPS73025DBVT, IC6 LP3990MF-1.2, IC7 TPS63000, IC8 ESP8266, IC9 SIM800C, Q1 IRLML6402, Q10 NTA4153NT1G, Q2 NTA4153NT1G, Q4 NTA4153NT1G, Q6 IRLML6402, Q7 16MHz, Q8 NTA4153NT1G, SW1 PWR, SW2 CAM, SW3 VOL+, SW4 VOL-, X1 MICROSIM, X10 AUDIO-JACKSMD, X13 OV2640, X14 EXT, X15 DF13-4P-1.25V, X2 BAT, X3 RM68120_LCD, X7 CTS, Y1 2.4Ghz, Y3 2.4Ghz, Y4 GSM_PCB, Y5 2.4Ghz

Commit message: fix charger schematic
Parts:
- removed C64, C65: 100n, netcat:R0402
- removed L7: 2.2uH, netcat:CDRH2D18LD
- removed R45, R46, R56: 10k, netcat:R0402
- C2: device netcat:SMC_A -> netcat:SMC_B
- moved C61 12.2 mm to (1.60, 49.7), turned to 270 degrees
- moved C2 11.2 mm to (7.80, 42.0)
- moved R35 9.55 mm to (16.1, 47.0), turned to 180 degrees
- moved R15 7.50 mm to (1.60, 44.0), turned to 90 degrees
- moved R57 6.14 mm to (7.20, 45.7), turned to 180 degrees
- moved R14 5.45 mm to (1.60, 47.0), turned to 90 degrees
- moved R22 5.14 mm to (7.20, 47.4), turned to 0 degrees
- moved R34 4.84 mm to (7.20, 49.1), turned to 0 degrees
- moved C72 4.47 mm to (11.4, 52.3), turned to 270 degrees
- moved Q1 2.07 mm to (18.3, 49.6), turned to 180 degrees
- moved IC22 1.58 mm to (11.8, 48.2), turned to 270 degrees
- moved R5 0.36 mm to (10.7, 37.8), turned to 0 degrees
- moved LED3 0.35 mm to (1.85, 40.5)
- moved R37 0.35 mm to (4.45, 40.5)
- moved Q8 0.10 mm to (13.3, 38.4)
Connections:
- removed net N$10: C64.1, IC22.6
- removed net N$28: IC22.25, IC22.26, L7.2
- removed net N$61: C65.1, IC22.10
- removed net N$87: IC22.16, R46.1, R56.1, X2.2
- removed net N$88: C72.2, IC22.9, R46.2
- net 3.3V: no longer IC22.5, IC22.7
- net GND: now also IC22.10, IC22.16, IC22.3, IC22.4; no longer C65.2, IC22.17, R45.1, R56.2
- net N$6: now also C72.2, IC22.5, IC22.7, IC22.9; no longer C64.2, IC22.27, IC22.28, L7.1
- net USB_CC1: no longer R45.2
- net V_USB: now also IC22.17; no longer IC22.3, IC22.4
Routing:
- net N$87: track 17.6 -> 0.00 mm, vias 1 -> 0
- net N$6: track 19.2 -> 6.75 mm, vias 2 -> 0
- net V_USB: track 43.7 -> 31.9 mm, vias 3 -> 1
- net 3.3V: track 787.1 -> 776.5 mm, vias 53 -> 50
- net N$88: track 9.60 -> 0.00 mm, vias 2 -> 0
- net BAT_CHG: track 41.8 -> 50.7 mm
- net V_SYS: track 33.0 -> 24.1 mm, vias 2 -> 0
- net V_BAT: track 8.51 -> 16.1 mm, vias 0 -> 1
- net N$28: track 7.49 -> 0.00 mm
- net PWR_OTG_MODE: track 52.4 -> 48.1 mm
- net GND: track 34.4 -> 38.6 mm, vias 450 -> 438
- net BAT_EN: track 10.1 -> 13.5 mm
- net N$61: track 2.62 -> 0.00 mm
- net N$10: track 2.59 -> 0.00 mm
- net V_INT: track 61.5 -> 59.4 mm
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
Commit message: fix mosfets
Parts:
- moved Q8 0.51 mm to (13.8, 38.3), turned to 180 degrees
- moved Q10 0.43 mm to (107.8, 24.9), turned to 270 degrees
- moved Q2 0.40 mm to (60.9, 35.2)
- moved Q4 0.25 mm to (62.8, 35.5), turned to 0 degrees
Routing:
- net GSM_PWRKEY: track 49.2 -> 47.0 mm
- net PWR_OTG_MODE: track 48.1 -> 46.4 mm
- net N$18: track 1.76 -> 2.89 mm

Commit message: added gnd holes for 3.3 dc-dc
Routing:
- net PWR_SHDN: track 61.4 -> 60.8 mm

Commit message: new modem dc-dc
Parts:
- removed C8: 100n, netcat:R0402
- removed C9: 220n, netcat:R0402
- removed L3: 2.2uH, netcat:CDRH2D18LD
- removed R10: 1M, netcat:R0402
- removed R11: 220k, netcat:R0402
- removed R52: 12k, netcat:R0402
- removed R58: 100k, netcat:R0402
- removed TP21: 4.0v, netcat:TP06R
- removed VD2: STPS0520Z, netcat:SOD123
- added L7: 2.2uH, netcat:CDRH2D18LD
- added R45: 100, netcat:R0402
- added R46: 1M, netcat:R0402
- C5: value 100n -> 10u; device netcat:R0402 -> netcat:SMC_B
- C6: value 100u -> 100n; device netcat:SMC_C -> netcat:R0402
- IC13: value MAX1708 -> TPS63001; device netcat:QSOP16 -> netcat:DFN10-3X3
- IC7: value TPS63000 -> TPS63001
- R51: value 27k -> 220k
- moved C6 8.65 mm to (50.8, 36.7), turned to 0 degrees
- moved TP19 6.47 mm to (24.6, 40.6)
- moved R51 5.04 mm to (50.8, 38.8)
- moved IC13 4.49 mm to (47.0, 36.7), turned to 270 degrees
- moved C5 3.83 mm to (43.3, 41.8), turned to 180 degrees
- moved C63 2.08 mm to (23.0, 40.0)
- moved R16 1.55 mm to (50.8, 34.2), turned to 180 degrees
- moved C1 1.06 mm to (20.8, 34.7), turned to 270 degrees
- moved C7 0.72 mm to (39.1, 34.3)
Connections:
- removed net N$12: IC7.10, R10.2, R11.1
- removed net N$15: IC13.3, IC13.4, IC13.5, L3.2, VD2.A
- removed net N$98: IC13.11, R51.1, R52.2
- new net N$10: C6.1, IC13.7, IC13.8, R45.1
- new net N$28: IC13.2, L7.2
- net !GSM_EN: now also IC13.6; no longer IC13.2
- net 3.3V: now also IC7.10; no longer R10.1
- net 4.0V: now also C5.+, IC13.1, R46.1; no longer C5.1, C6.+, IC13.10, IC13.16, R51.2, TP21.TP, VD2.C
- net GND: now also C5.-, C6.2, IC13.3, IC13.PPAD, R51.2; no longer C5.2, C6.-, C8.2, C9.2, IC13.12, IC13.13, IC13.14, IC13.15, IC13.6, R11.2, R52.1, R58.2
- net N$19: now also IC13.10, R46.2, R51.1; no longer C8.1, IC13.7, R58.1
- net N$20: now also IC13.4, L7.1; no longer C9.1, IC13.8
- net V_INT: now also IC13.5, R45.2; no longer IC13.1, L3.1
Routing:
- net 4.0V: track 50.6 -> 37.1 mm
- net N$15: track 13.1 -> 0.00 mm
- net V_INT: track 59.4 -> 67.8 mm
- net N$10: track 0.00 -> 4.22 mm
- net N$12: track 4.05 -> 0.00 mm
- net N$28: track 0.00 -> 3.89 mm
- net N$98: track 3.35 -> 0.00 mm
- net N$20: track 1.57 -> 3.37 mm
- net 3.3V: track 776.5 -> 778.1 mm
- net N$19: track 2.84 -> 4.40 mm
- net !GSM_EN: track 33.2 -> 34.4 mm
- net GND: vias 438 -> 436

Commit message: fix size of pads on speaker
Routing:
- net SPKRP: track 46.6 -> 45.7 mm
- net GND: vias 436 -> 439
Changed lines of the file:
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@@
 <setting verticaltext="up"/>
 </settings>
-<grid distance="0.05" unitdist="mm" unit="mm" style="lines" multiple="1" display="yes" altdistance="1" altunitdist="mm" altunit="mm"/>
+<grid distance="0.1" unitdist="mm" unit="mm" style="lines" multiple="1" display="yes" altdistance="1" altunitdist="mm" altunit="mm"/>
 <layers>
 <layer number="1" name="Top" color="4" fill="1" visible="yes" active="yes"/>
@@
 <layer number="40" name="bKeepout" color="1" fill="11" visible="no" active="yes"/>
 <layer number="41" name="tRestrict" color="4" fill="10" visible="yes" active="yes"/>
-<layer number="42" name="bRestrict" color="1" fill="10" visible="no" active="yes"/>
+<layer number="42" name="bRestrict" color="1" fill="10" visible="yes" active="yes"/>
 <layer number="43" name="vRestrict" color="2" fill="10" visible="no" active="yes"/>
 <layer number="44" name="Drills" color="7" fill="1" visible="no" active="yes"/>
@@
 <rectangle x1="116" y1="30" x2="116.1" y2="36.4" layer="41"/>
 <rectangle x1="116" y1="37" x2="116.1" y2="41" layer="41"/>
-<rectangle x1="116" y1="30" x2="116.1" y2="37.45" layer="42"/>
 <rectangle x1="82" y1="53" x2="82.1" y2="54.2" layer="41"/>
 <rectangle x1="82" y1="54.9" x2="82.1" y2="56" layer="41"/>
@@
 <rectangle x1="12.3" y1="50" x2="12.55" y2="50.05" layer="41" rot="R90"/>
 <rectangle x1="11.9" y1="50" x2="12.15" y2="50.05" layer="41" rot="R90"/>
+<rectangle x1="116" y1="30" x2="116.1" y2="38.95" layer="42"/>
 </plain>
 <attributes>
@@
 <via x="40.25" y="29.6" extent="1-16" drill="0.3048" shape="octagon"/>
 <via x="77.4" y="23.1" extent="1-16" drill="0.3048" shape="octagon"/>
-<via x="63.75" y="30.05" extent="1-16" drill="0.3048" shape="octagon"/>
+<via x="64" y="30.05" extent="1-16" drill="0.3048" shape="octagon"/>
 <via x="29.8" y="26.05" extent="1-16" drill="0.3048" shape="octagon"/>
 <via x="64.75" y="8.95" extent="1-16" drill="0.3048" shape="octagon"/>
@@
 <via x="82.2" y="20.3" extent="1-16" drill="0.3048" shape="octagon"/>
 <via x="113.4" y="41.2" extent="1-16" drill="0.3048" shape="octagon"/>
-<via x="113.4" y="39.8" extent="1-16" drill="0.3048" shape="octagon"/>
+<via x="113.4" y="39.2" extent="1-16" drill="0.3048" shape="octagon"/>
 <via x="113.4" y="37.8" extent="1-16" drill="0.3048" shape="octagon"/>
 <contactref element="C71" pad="2"/>
@@
 <via x="41.85" y="36.65" extent="1-16" drill="0.3048" shape="octagon"/>
 <via x="44" y="36.45" extent="1-16" drill="0.3048" shape="octagon"/>
+<via x="45.05" y="31.2" extent="1-16" drill="0.3048" shape="octagon"/>
+<via x="53.1" y="33.1" extent="1-16" drill="0.3048" shape="octagon"/>
+<via x="63.2" y="30.05" extent="1-16" drill="0.3048" shape="octagon"/>
 </signal>
 <signal name="SDHC_ST">
@@
 <via x="100.25" y="15" extent="1-16" drill="0.3048" shape="octagon"/>
 <contactref element="B2" pad="1"/>
-<wire x1="114.65" y1="38.2" x2="115.125" y2="38.675" width="0.2" layer="16"/>
-<wire x1="115.125" y1="38.675" x2="115.5" y2="39.05" width="0.2" layer="16"/>
 <wire x1="106.25" y1="22.2" x2="100.25" y2="16.2" width="0.2" layer="16"/>
 <wire x1="100.25" y1="16.2" x2="100.25" y2="15" width="0.2" layer="16"/>
 <wire x1="113.5" y1="24.25" x2="113.5" y2="31.6" width="0.2" layer="16"/>
-<wire x1="112.65" y1="39.15" x2="115.125" y2="39.15" width="0.2" layer="16"/>
-<wire x1="115.125" y1="39.15" x2="115.125" y2="38.675" width="0.2" layer="16"/>
 <wire x1="106.25" y1="22.2" x2="110.7" y2="22.2" width="0.2" layer="16"/>
 <wire x1="110.7" y1="22.2" x2="112.35" y2="23.85" width="0.2" layer="16"/>
@@
 <wire x1="113.1" y1="23.85" x2="113.5" y2="24.25" width="0.2" layer="16"/>
 <wire x1="113.5" y1="31.6" x2="110.95" y2="34.15" width="0.2" layer="16"/>
-<wire x1="110.95" y1="34.15" x2="110.95" y2="37.45" width="0.2" layer="16"/>
-<wire x1="110.95" y1="37.45" x2="112.65" y2="39.15" width="0.2" layer="16"/>
+<wire x1="110.95" y1="34.15" x2="110.95" y2="37.75" width="0.2" layer="16"/>
+<wire x1="110.95" y1="37.75" x2="113" y2="39.8" width="0.2" layer="16"/>
 <wire x1="94.4" y1="15" x2="100.25" y2="15" width="0.2" layer="1"/>
 <wire x1="94.4" y1="15" x2="93.69" y2="15.71" width="0.2" layer="1"/>
 <wire x1="93.69" y1="15.71" x2="92.59" y2="15.71" width="0.2" layer="1"/>
+<wire x1="113" y1="39.8" x2="115.5" y2="39.8" width="0.2" layer="16"/>
 </signal>
 <signal name="SPKRN">
@@
 <wire x1="112.55" y1="23.35" x2="113.3" y2="23.35" width="0.2" layer="16"/>
 <wire x1="113.3" y1="23.35" x2="114.15" y2="24.2" width="0.2" layer="16"/>
-<wire x1="114.15" y1="24.2" x2="114.15" y2="25.7" width="0.2" layer="16"/>
-<wire x1="114.15" y1="25.7" x2="115.5" y2="27.05" width="0.2" layer="16"/>
 <wire x1="99.7" y1="15.4" x2="99.95" y2="15.65" width="0.2" layer="1"/>
 <wire x1="99.95" y1="15.65" x2="100.95" y2="15.65" width="0.2" layer="1"/>
 <wire x1="93.89" y1="16.11" x2="92.59" y2="16.11" width="0.2" layer="1"/>
+<wire x1="114.15" y1="24.2" x2="114.15" y2="26.3" width="0.2" layer="16"/>
+<wire x1="114.15" y1="26.3" x2="115.5" y2="26.3" width="0.2" layer="16"/>
 </signal>
 <signal name="RINGP">

Commit message: fix VDD_RTC on wifi chip
Connections:
- net 3.3V: no longer IC8.5
Routing:
- net 3.3V: track 778.1 -> 777.1 mm
Changed lines of the file:
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@@
 <grid distance="0.1" unitdist="mm" unit="mm" style="lines" multiple="1" display="yes" altdistance="1" altunitdist="mm" altunit="mm"/>
 <layers>
-<layer number="1" name="Top" color="4" fill="1" visible="yes" active="yes"/>
+<layer number="1" name="Top" color="4" fill="1" visible="no" active="yes"/>
 <layer number="2" name="Route2" color="1" fill="3" visible="no" active="no"/>
 <layer number="3" name="Route3" color="4" fill="3" visible="no" active="no"/>
@@
 <layer number="14" name="Route14" color="1" fill="6" visible="no" active="no"/>
 <layer number="15" name="Route15" color="4" fill="6" visible="no" active="no"/>
-<layer number="16" name="Bottom" color="1" fill="1" visible="no" active="yes"/>
+<layer number="16" name="Bottom" color="1" fill="1" visible="yes" active="yes"/>
 <layer number="17" name="Pads" color="2" fill="1" visible="yes" active="yes"/>
 <layer number="18" name="Vias" color="2" fill="1" visible="yes" active="yes"/>
 <layer number="19" name="Unrouted" color="6" fill="1" visible="yes" active="yes"/>
 <layer number="20" name="Dimension" color="15" fill="1" visible="yes" active="yes"/>
-<layer number="21" name="tPlace" color="7" fill="1" visible="yes" active="yes"/>
-<layer number="22" name="bPlace" color="7" fill="1" visible="no" active="yes"/>
-<layer number="23" name="tOrigins" color="15" fill="1" visible="yes" active="yes"/>
-<layer number="24" name="bOrigins" color="15" fill="1" visible="no" active="yes"/>
+<layer number="21" name="tPlace" color="7" fill="1" visible="no" active="yes"/>
+<layer number="22" name="bPlace" color="7" fill="1" visible="yes" active="yes"/>
+<layer number="23" name="tOrigins" color="15" fill="1" visible="no" active="yes"/>
+<layer number="24" name="bOrigins" color="15" fill="1" visible="yes" active="yes"/>
 <layer number="25" name="tNames" color="7" fill="1" visible="no" active="yes"/>
 <layer number="26" name="bNames" color="7" fill="1" visible="no" active="yes"/>
@@
 <layer number="49" name="Reference" color="7" fill="1" visible="no" active="yes"/>
 <layer number="50" name="dxf" color="7" fill="1" visible="no" active="no"/>
-<layer number="51" name="tDocu" color="7" fill="1" visible="yes" active="yes"/>
-<layer number="52" name="bDocu" color="7" fill="1" visible="no" active="yes"/>
+<layer number="51" name="tDocu" color="7" fill="1" visible="no" active="yes"/>
+<layer number="52" name="bDocu" color="7" fill="1" visible="yes" active="yes"/>
 <layer number="53" name="tGND_GNDA" color="7" fill="9" visible="no" active="no"/>
 <layer number="54" name="bGND_GNDA" color="1" fill="9" visible="no" active="no"/>
@@
 <contactref element="IC8" pad="11"/>
 <contactref element="IC8" pad="17"/>
-<contactref element="IC8" pad="5"/>
 <wire x1="105.25" y1="52.95" x2="105.25" y2="53.65" width="0.2" layer="1"/>
 <wire x1="108.1" y1="50.9" x2="107.3" y2="50.9" width="0.2" layer="1"/>
 <wire x1="107.3" y1="51.4" x2="108.6" y2="51.4" width="0.2" layer="1"/>
 <wire x1="103.25" y1="47.7" x2="103.25" y2="48.35" width="0.2" layer="1"/>
-<wire x1="104.75" y1="52.95" x2="104.75" y2="53.65" width="0.2" layer="1"/>
-<wire x1="104.75" y1="53.65" x2="105.25" y2="53.65" width="0.2" layer="1"/>
 <wire x1="105.75" y1="52.95" x2="105.75" y2="53.65" width="0.2" layer="1"/>
 <wire x1="105.75" y1="53.65" x2="105.25" y2="53.65" width="0.2" layer="1"/>
@@
 <wire x1="107.95" y1="54.35" x2="104.75" y2="54.35" width="0.4064" layer="16"/>
 <wire x1="108.3" y1="54.7" x2="107.95" y2="54.35" width="0.2" layer="1"/>
-<wire x1="104.75" y1="54.35" x2="104.75" y2="53.65" width="0.2" layer="1"/>
 <wire x1="106.75" y1="52.95" x2="106.75" y2="53.4" width="0.2" layer="1"/>
 <wire x1="106.75" y1="53.4" x2="106.95" y2="53.6" width="0.2" layer="1"/>
@@
 <wire x1="17.95" y1="47" x2="19.05" y2="45.9" width="0.2" layer="1"/>
 <contactref element="IC7" pad="10"/>
-<wire x1="23" y1="40.6" x2="22.6" y2="40.6" width="0.2" layer="1"/>
-<wire x1="22.6" y1="40.6" x2="20.75" y2="40.6" width="0.2" layer="1"/>
+<wire x1="23" y1="40.6" x2="20.75" y2="40.6" width="0.2" layer="1"/>
 <wire x1="24.55" y1="39.45" x2="24.55" y2="40.6" width="0.2" layer="1"/>
 <wire x1="24.55" y1="40.6" x2="23" y2="40.6" width="0.2" layer="1"/>
@@
 <wire x1="20.8" y1="36" x2="20.75" y2="36.2" width="0.3048" layer="1"/>
 <wire x1="20.75" y1="39.1" x2="20.75" y2="36.2" width="0.4064" layer="1"/>
+<wire x1="105.25" y1="53.65" x2="104.75" y2="54.15" width="0.2" layer="1"/>
+<wire x1="104.75" y1="54.15" x2="104.75" y2="54.35" width="0.2" layer="1"/>
 </signal>
 <signal name="AQ13">
@@
 <wire x1="52.01" y1="37.9" x2="49.52" y2="40.39" width="0.2" layer="16"/>
 <contactref element="IC8" pad="7"/>
-<wire x1="103.75" y1="52.95" x2="103.75" y2="53.8" width="0.2" layer="1"/>
 <via x="103.75" y="53.8" extent="1-16" drill="0.3048" shape="octagon"/>
 <wire x1="94.15" y1="49.65" x2="93.3" y2="48.8" width="0.2" layer="16"/>
@@
 <wire x1="39.41" y1="38.56" x2="41.24" y2="40.39" width="0.2" layer="16"/>
 <wire x1="41.24" y1="40.39" x2="49.52" y2="40.39" width="0.2" layer="16"/>
+<wire x1="103.75" y1="52.95" x2="103.75" y2="53.8" width="0.2" layer="1"/>
 </signal>
 <signal name="ESP_TX">

Commit message: new pkg of wifi's crystall
Parts:
- OSC1: device netcat:CRYSTAL_MINI_26 -> netcat:CRYSTAL_MICRO_26
- moved OSC1 0.16 mm to (110.8, 49.8)
- moved Q1 0.15 mm to (18.3, 49.8)
Routing:
- net SD_CLK: track 12.5 -> 9.80 mm
- net GND: track 38.6 -> 37.3 mm, vias 439 -> 444
- net N$27: track 5.10 -> 5.82 mm

Commit message: new 1.2/2.5 dc-dc, fix bad pinout on audiocodec
Parts:
- removed C10, C78: 100n, netcat:R0402
- C7: device netcat:SMC_C -> netcat:SMC_B
- IC5: value TPS73025DBVT -> LP3990TL; device netcat:SOT23-5 -> netcat:DSBGA
- IC6: value LP3990MF-1.2 -> LP3990TL; device netcat:SOT23-5 -> netcat:DSBGA
- moved IC6 12.9 mm to (36.4, 41.9), turned to 180 degrees
- moved C4 8.59 mm to (34.6, 41.8)
- moved IC5 5.57 mm to (39.6, 41.9), turned to 180 degrees
- moved C5 3.35 mm to (46.6, 41.9), turned to 0 degrees
- moved C29 3.08 mm to (42.5, 41.5)
- moved C28 2.28 mm to (31.2, 43.5), turned to 180 degrees
- moved C3 2.06 mm to (37.9, 41.7), turned to 270 degrees
- moved L7 1.03 mm to (42.5, 34.5)
- moved C7 0.75 mm to (39.1, 33.5)
Connections:
- removed net N$100: C78.1, IC6.4
- removed net N$21: C10.1, IC5.4
- net 1.2V: now also IC6.B1; no longer IC6.5
- net 2.5V: now also IC5.B1; no longer IC5.5
- net 3.3V: now also IC18.24, IC18.40; no longer IC18.23, IC18.38
- net EE_I2C_SCL: now also IC18.37; no longer IC18.36
- net EE_I2C_SDA: now also IC18.36; no longer IC18.35
- net GND: now also IC18.12, IC18.17, IC18.20, IC18.26, IC5.A1, IC6.A1; no longer C10.2, C78.2, IC18.16, IC18.19, IC18.25, IC18.40, IC5.2, IC6.2
- net GSM_A_IN: now also IC18.21; no longer IC18.20
- net MIC_PWR: now also IC18.29; no longer IC18.28
- net N$46: now also IC18.13; no longer IC18.12
- net N$48: now also IC18.18; no longer IC18.17
- net N$49: now also IC18.31; no longer IC18.30
- net N$50: now also IC18.25; no longer IC18.24
- net N$58: now also IC18.15; no longer IC18.14
- net N$59: now also IC18.14; no longer IC18.13
- net N$60: now also IC18.19; no longer IC18.18
- net N$62: now also IC18.35; no longer IC18.34
- net N$63: now also IC18.32; no longer IC18.31
- net N$64: now also IC18.34; no longer IC18.33
- net N$70: now also IC18.16; no longer IC18.15
- net RINGN: now also IC18.27; no longer IC18.26
- net RINGP: now also IC18.28; no longer IC18.27
- net SPKRN: now also IC18.23; no longer IC18.22
- net SPKRP: now also IC18.22; no longer IC18.21
- net V_INT: now also IC5.A2, IC5.B2, IC6.A2, IC6.B2; no longer IC5.1, IC5.3, IC6.1, IC6.3
Routing:
- net 1.2V: track 186.5 -> 176.2 mm
- net SDIO0: track 26.7 -> 29.3 mm
- net N$100: track 2.12 -> 0.00 mm
- net N$21: track 1.73 -> 0.00 mm
- net N$49: track 3.10 -> 4.49 mm
- net V_INT: track 67.9 -> 66.7 mm
- net 2.5V: track 143.7 -> 144.8 mm
- net GSM_A_IN: track 42.9 -> 42.3 mm
- net N$28: track 3.89 -> 3.33 mm
- net N$48: track 36.9 -> 36.4 mm
- net GND: vias 444 -> 438
