File: redphone.brd (EAGLE design)
At the start: 139 x 65 mm, 233 parts, among them IC1 EP4CE15E22, IC10 74LVC1G02DCK, IC11 74LVC1G02DCK, IC12 74LVC1G02DCK, IC13 TPS63001, IC15 LSM303DLHC, IC16 EPCS4SI8N, IC17 L3GD20, IC18 WM8903, IC19 AT25SF041, IC2 STM32F429ZIT, IC20 MP34DT01, IC21 PT4181, IC22 MAX8903A, IC23 NRF24L01+, IC24 BME280, IC25 APDS-9960, IC3 MT48LC16M16A2TG, IC4 MAX8815A, IC5 LP3990TL, IC6 LP3990TL, IC7 TPS63001, IC8 ESP8266, IC9 SIM800C, Q1 IRLML6402, Q10 NTA4153NT1G, Q2 NTA4153NT1G, Q4 NTA4153NT1G, Q6 IRLML6402, Q7 16MHz, Q8 NTA4153NT1G, SW1 PWR, SW2 CAM, SW3 VOL+, SW4 VOL-, X1 MICROSIM, X10 AUDIO-JACKSMD, X13 OV2640, X14 EXT, X15 DF13-4P-1.25V, X2 BAT, X3 RM68120_LCD, X7 CTS, Y1 2.4Ghz, Y3 2.4Ghz, Y4 GSM_PCB, Y5 2.4Ghz

Commit message: i2c & cts tps, cap pkg fix, names fix, route fix
Parts:
- added TP21: AIN, netcat:TP06R
- added TP23: AOUT, netcat:TP06R
- added TP24: TSI, netcat:TP06R
- added TP25: MSDA, netcat:TP06R
- added TP26: MSCL, netcat:TP06R
- C1, C2, C5, C7: device netcat:SMC_B -> netcat:SMC_A
- IC1: value EP4CE15E22 -> EP4CE6E22
- IC13: value TPS63001 -> TPS63000
- IC14: value (none) -> 24LC256
- IC23: device netcat:QFN20_ALT1 -> netcat:QFN20
- moved TP10 1.14 mm to (68.8, 4.50)
Connections:
- net EE_I2C_SCL: now also TP26.TP
- net EE_I2C_SDA: now also TP25.TP
- net GSM_A_IN: now also TP21.TP
- net GSM_A_OUT: now also TP23.TP
- net TS_INT: now also TP24.TP
Routing:
- net EE_I2C_SCL: track 152.7 -> 162.4 mm, vias 6 -> 7
- net EE_I2C_SDA: track 148.7 -> 156.7 mm, vias 7 -> 8
- net GSM_A_OUT: track 40.7 -> 42.0 mm
- net FPGA_SCL: track 44.6 -> 43.5 mm
- net TS_INT: track 50.0 -> 50.8 mm
- net GSM_A_IN: track 42.3 -> 42.9 mm
- net GND: vias 438 -> 437
Other:
- board size 139 x 65 mm -> 122 x 65 mm

Commit message: connect rtc to vbat, change mosfet type
Parts:
- removed X15: DF13-4P-1.25V, netcat:DF13C-4P-1.25V
- added C8: 1u, netcat:R0603
- added VD2: STPS0520Z, netcat:SOD123
- Q1, Q6: value IRLML6402 -> IRLML2502
- moved OSC3 3.40 mm to (18.5, 3.60)
- moved C34 3.39 mm to (19.9, 1.65), turned to 90 degrees
- moved C35 3.19 mm to (17.1, 1.60), turned to 90 degrees
- moved C33 2.42 mm to (26.8, 3.45)
- moved OSC2 2.29 mm to (24.1, 3.15)
- moved C32 2.13 mm to (21.6, 2.85)
- moved R26 1.97 mm to (28.0, 3.45), turned to 90 degrees
- moved C62 1.17 mm to (29.2, 3.45), turned to 90 degrees
Connections:
- new net N$12: C8.1, IC2.6, VD2.C
- net 3.3V: no longer IC2.6, X15.2
- net FPGA_RX: no longer X15.4
- net FPGA_TX: no longer X15.3
- net GND: now also C8.2; no longer X15.1
- net V_BAT: now also VD2.A
Routing:
- net V_BAT: track 16.1 -> 71.7 mm, vias 1 -> 2
- net N$12: track 0.00 -> 7.27 mm
- net OSC32O: track 8.59 -> 5.11 mm
- net 3.3V: track 776.8 -> 773.6 mm
- net FPGA_TX: track 50.9 -> 48.1 mm
- net OSCI: track 8.80 -> 7.22 mm
- net OSCO: track 6.04 -> 4.48 mm
- net BL_RST: track 2.99 -> 4.46 mm
- net BAT_SENS: track 58.1 -> 57.0 mm
- net FPGA_RX: track 49.0 -> 48.2 mm
- net RINGP: track 171.8 -> 172.6 mm
- net SL_BOOT0: track 21.5 -> 22.1 mm
- net RINGN: track 186.1 -> 186.8 mm
- net OSC32I: track 6.99 -> 6.40 mm
- net UART_EXT_RX: track 47.5 -> 48.1 mm
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
Commit message: swap usb_cc1 to mcu_rst
Connections:
- removed net USB_CC1: IC2.110, X16.A5
- net BL_RST: now also X16.A5
Routing:
- net BL_RST: track 4.46 -> 65.3 mm, vias 0 -> 4
- net USB_CC1: track 19.5 -> 0.00 mm, vias 2 -> 0
- net RINGN: track 186.8 -> 186.2 mm
- net GND: vias 436 -> 440

Commit message: move ts connector
Parts:
- moved X7 1.10 mm to (94.2, 50.7)
Routing:
- net TS_SCL: track 51.5 -> 55.0 mm, vias 2 -> 4
- net 3.3V: track 773.6 -> 775.0 mm
- net TS_INT: track 50.8 -> 51.9 mm
- net TS_SDA: track 51.4 -> 52.5 mm
Other:
- outline, holes or cut-outs redrawn

Commit message: change fpga crystal to osc, update lbr
Parts:
- removed C53: 22p, netcat:R0402
- C54: value 22p -> 100n
- OSC1: value 26 Mhz -> 26 MHz; device netcat:CRYSTAL_MICRO_26 -> netcat:2520
- OSC2, Q7: device netcat:CRYSTAL_MINI_26 -> netcat:3225
- OSC3: device netcat:CRYSTAL_MICRO_32 -> netcat:3215
- OSC4: value 48 mhz -> 48 MHz; device netcat:CRYSTAL_MINI_26 -> netcat:3225
- moved C54 0.47 mm to (63.2, 32.4)
Connections:
- removed net OSCO1: C54.2, IC1.25, OSC4.1
- net 3.3V: now also C54.1, OSC4.4
- net GND: now also C54.2; no longer C53.1, C54.1, OSC4.4
- net OSCI1: no longer C53.2
Routing:
- net 3.3V: track 775.0 -> 781.8 mm
- net OSCO1: track 3.66 -> 0.00 mm
- net OSCI1: track 6.19 -> 4.98 mm
Changed lines of the file:
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@@
 <layer number="23" name="tOrigins" color="15" fill="1" visible="yes" active="yes"/>
 <layer number="24" name="bOrigins" color="15" fill="1" visible="no" active="yes"/>
-<layer number="25" name="tNames" color="7" fill="1" visible="no" active="yes"/>
+<layer number="25" name="tNames" color="7" fill="1" visible="yes" active="yes"/>
 <layer number="26" name="bNames" color="7" fill="1" visible="no" active="yes"/>
 <layer number="27" name="tValues" color="7" fill="1" visible="no" active="yes"/>
@@
 <attribute name="VALUE" x="110.115" y="45.4625" size="0.8128" layer="27" font="vector"/>
 </element>
-<element name="OSC1" library="netcat" package="CRYSTAL_MICRO_26" value="26 Mhz" x="110.8" y="49.8" smashed="yes" rot="R270">
+<element name="OSC1" library="netcat" package="2520" value="26 MHz" x="110.8" y="49.8" smashed="yes" rot="R270">
 <attribute name="VALUE" x="113.992" y="50.886" size="0.8128" layer="27" font="vector" ratio="10" rot="R270"/>
 <attribute name="NAME" x="109.593" y="48.484" size="0.8128" layer="25" font="vector" rot="R90"/>
@@
 <attribute name="VALUE" x="112.835" y="54.482" size="0.8128" layer="27" font="vector" rot="R180"/>
 </element>
-<element name="Q7" library="netcat" package="CRYSTAL_MINI_26" value="16MHz" x="106.66" y="30.51" smashed="yes" rot="R180">
+<element name="Q7" library="netcat" package="3225" value="16MHz" x="106.66" y="30.51" smashed="yes" rot="R180">
 <attribute name="VALUE" x="107.746" y="27.318" size="0.8128" layer="27" font="vector" ratio="10" rot="R180"/>
 <attribute name="NAME" x="107.376" y="28.728" size="0.8128" layer="25" font="vector" rot="R180"/>
@@
 <attribute name="VALUE" x="35.73488125" y="29.827646875" size="0.8128" layer="27" font="vector" rot="R135"/>
 </element>
-<element name="OSC2" library="netcat" package="CRYSTAL_MINI_26" value="8 mhz" x="24.15" y="3.15" smashed="yes" rot="R180">
+<element name="OSC2" library="netcat" package="3225" value="8 mhz" x="24.15" y="3.15" smashed="yes" rot="R180">
 <attribute name="NAME" x="22.76" y="4.8075" size="0.8128" layer="25" font="vector" ratio="10"/>
 <attribute name="VALUE" x="26.436" y="3.658" size="0.8128" layer="27" font="vector" ratio="10" rot="R180"/>
@@
 <attribute name="VALUE" x="10.932" y="2.665" size="0.8128" layer="27" font="vector" rot="R90"/>
 </element>
-<element name="OSC3" library="netcat" package="CRYSTAL_MICRO_32" value="32.768k" x="18.5" y="3.6" smashed="yes">
+<element name="OSC3" library="netcat" package="3215" value="32.768k" x="18.5" y="3.6" smashed="yes">
 <attribute name="NAME" x="17.08" y="4.5075" size="0.8128" layer="25" font="vector" ratio="10"/>
 <attribute name="VALUE" x="16.214" y="4.362" size="0.8128" layer="27" font="vector" ratio="10"/>
@@
 <attribute name="VALUE" x="97.039" y="21.9645" size="0.8128" layer="27" font="vector" rot="R180"/>
 </element>
-<element name="OSC4" library="netcat" package="CRYSTAL_MINI_26" value="48 mhz" x="65.9" y="32" smashed="yes">
-<attribute name="NAME" x="64.46" y="29.6075" size="0.8128" layer="25" font="vector" ratio="10"/>
-<attribute name="VALUE" x="63.614" y="31.492" size="0.8128" layer="27" font="vector" ratio="10"/>
-</element>
-<element name="C53" library="netcat" package="R0402" value="22p" x="66.5" y="34.15" smashed="yes">
-<attribute name="NAME" x="65.165" y="34.962" size="0.8128" layer="25" font="vector"/>
-<attribute name="VALUE" x="65.865" y="32.118" size="0.8128" layer="27" font="vector"/>
-</element>
-<element name="C54" library="netcat" package="R0402" value="22p" x="63.4" y="31.9" smashed="yes" rot="R270">
-<attribute name="NAME" x="62.738" y="30.915" size="0.8128" layer="25" font="vector" rot="R90"/>
-<attribute name="VALUE" x="61.368" y="32.535" size="0.8128" layer="27" font="vector" rot="R270"/>
+<element name="C54" library="netcat" package="R0402" value="100n" x="63.25" y="32.35" smashed="yes" rot="R270">
+<attribute name="NAME" x="62.588" y="31.215" size="0.8128" layer="25" font="vector" rot="R90"/>
+<attribute name="VALUE" x="61.218" y="32.985" size="0.8128" layer="27" font="vector" rot="R270"/>
 </element>
 <element name="C55" library="netcat" package="R0402" value="100n" x="38.05" y="16.9" smashed="yes" rot="R270">
@@
 <element name="Y4" library="netcat" package="GSM_ANT" value="GSM_PCB" x="60.05" y="62.95"/>
 <element name="Q4" library="netcat" package="SOT-416" value="NTA4153NT1G" x="62.8" y="35.5" smashed="yes">
-<attribute name="NAME" x="64.455" y="34.345" size="0.8128" layer="25" font="vector" rot="R180"/>
+<attribute name="NAME" x="64.355" y="34.345" size="0.8128" layer="25" font="vector" rot="R180"/>
 <attribute name="VALUE" x="60.895" y="32.325" size="0.8128" layer="27" font="vector"/>
 </element>
@@
 <attribute name="VALUE" x="15.189" y="2.6645" size="0.8128" layer="27" font="vector" rot="R180"/>
 </element>
+<element name="OSC4" library="netcat" package="3225" value="48 MHz" x="65.9" y="32.05" smashed="yes">
+<attribute name="VALUE" x="64.814" y="35.242" size="0.8128" layer="27" font="vector" ratio="10"/>
+<attribute name="NAME" x="64.884" y="33.932" size="0.8128" layer="25" font="vector"/>
+</element>
 </elements>
 <signals>
@@
 <contactref element="IC9" pad="12"/>
 <contactref element="IC9" pad="10"/>
-<contactref element="OSC4" pad="4"/>
-<contactref element="OSC4" pad="2"/>
-<contactref element="C53" pad="1"/>
-<contactref element="C54" pad="1"/>
 <polygon width="0.2" layer="1" isolate="0.2">
 <vertex x="0" y="0"/>
@@
 <via x="62.25" y="52.25" extent="1-16" drill="0.3048" shape="octagon"/>
 <via x="78.75" y="52.25" extent="1-16" drill="0.3048" shape="octagon"/>
-<via x="64.65" y="34.1" extent="1-16" drill="0.3048" shape="octagon"/>
+<via x="64.45" y="34.35" extent="1-16" drill="0.3048" shape="octagon"/>
 <via x="78.35" y="34.25" extent="1-16" drill="0.3048" shape="octagon"/>
 <via x="90.9" y="43.05" extent="1-16" drill="0.3048" shape="octagon"/>
@@
 <via x="1.5" y="6" extent="1-16" drill="0.8" diameter="1.55" shape="octagon"/>
 <via x="7.5" y="6" extent="1-16" drill="0.8" diameter="1.55" shape="octagon"/>
+<contactref element="OSC4" pad="2"/>
+<contactref element="C54" pad="2"/>
 </signal>
 <signal name="SDHC_ST">
@@
 <wire x1="98" y1="50.2" x2="97.25" y2="50.95" width="0.2" layer="1"/>
 <wire x1="97.25" y1="50.95" x2="93.71" y2="50.95" width="0.2" layer="1"/>
+<contactref element="C54" pad="1"/>
+<contactref element="OSC4" pad="4"/>
+<wire x1="64.25" y1="28.75" x2="64.25" y2="29.4" width="0.2" layer="1"/>
+<wire x1="64.25" y1="29.4" x2="64.7" y2="29.85" width="0.2" layer="1"/>
+<wire x1="64.7" y1="29.85" x2="65" y2="29.85" width="0.2" layer="1"/>
+<wire x1="65" y1="29.85" x2="65.55" y2="30.4" width="0.2" layer="1"/>
+<wire x1="65.55" y1="30.4" x2="65.55" y2="32.0675" width="0.2" layer="1"/>
+<wire x1="65.55" y1="32.0675" x2="64.62" y2="32.9975" width="0.2" layer="1"/>
+<wire x1="63.25" y1="33" x2="64.6175" y2="33" width="0.2" layer="1"/>
+<wire x1="64.6175" y1="33" x2="64.62" y2="32.9975" width="0.2" layer="1"/>
 </signal>
 <signal name="AQ13">
@@
 </signal>
 <signal name="OSCI1">
-<contactref element="C53" pad="2"/>
-<contactref element="OSC4" pad="3"/>
 <contactref element="IC1" pad="24"/>
-<wire x1="65.25" y1="28.75" x2="65.25" y2="30.1" width="0.2" layer="1"/>
-<wire x1="65.25" y1="30.1" x2="65.85" y2="30.7" width="0.2" layer="1"/>
-<wire x1="65.85" y1="30.7" x2="65.85" y2="31.77625" width="0.2" layer="1"/>
-<wire x1="65.85" y1="31.77625" x2="67.02125" y2="32.9475" width="0.2" layer="1"/>
-<wire x1="67.15" y1="34.15" x2="67.15" y2="33.07625" width="0.2" layer="1"/>
-<wire x1="67.15" y1="33.07625" x2="67.02125" y2="32.9475" width="0.2" layer="1"/>
-</signal>
-<signal name="OSCO1">
-<contactref element="OSC4" pad="1"/>
-<contactref element="C54" pad="2"/>
-<contactref element="IC1" pad="25"/>
-<wire x1="64.75" y1="28.75" x2="64.75" y2="30.9225" width="0.2" layer="1"/>
-<wire x1="64.75" y1="30.9225" x2="64.62" y2="31.0525" width="0.2" layer="1"/>
-<wire x1="63.4" y1="31.25" x2="64.4225" y2="31.25" width="0.2" layer="1"/>
-<wire x1="64.4225" y1="31.25" x2="64.62" y2="31.0525" width="0.2" layer="1"/>
+<contactref element="OSC4" pad="3"/>
+<wire x1="65.25" y1="28.75" x2="65.25" y2="29.5" width="0.2" layer="1"/>
+<wire x1="65.25" y1="29.5" x2="66.1" y2="30.35" width="0.2" layer="1"/>
+<wire x1="66.1" y1="30.35" x2="66.1" y2="32.07625" width="0.2" layer="1"/>
+<wire x1="66.1" y1="32.07625" x2="67.02125" y2="32.9975" width="0.2" layer="1"/>
 </signal>
 <signal name="JACK_MIC">

Commit message: lowdrop en ctrl from stm
Parts:
- removed SCL1: PB12, netcat:TP06R
- VD2: value STPS0520Z -> BAS516; device netcat:SOD123 -> netcat:SOD523
- moved C8 1.88 mm to (13.5, 2.65)
- moved VD2 1.40 mm to (13.5, 1.10)
- moved LOGO1 0.25 mm to (52.0, 0.53)
Connections:
- removed net N$95: IC2.73, SCL1.TP
- new net FPGA_EN: IC2.73, IC5.A2, IC6.A2
- net V_INT: no longer IC5.A2, IC6.A2
Routing:
- net FPGA_EN: track 0.00 -> 27.0 mm, vias 0 -> 3
- net N$95: track 3.13 -> 0.00 mm
- net V_INT: track 66.7 -> 64.2 mm
- net N$12: track 7.27 -> 8.28 mm
- net EE_I2C_SCL: track 162.4 -> 161.5 mm
- net EE_I2C_SDA: track 156.7 -> 156.0 mm
- net GND: vias 440 -> 439

Commit message: added ds18b20, udfn pack for eeprom, some route fix
Parts:
- removed TP13: TSCL, netcat:TP06R
- removed TP25: MSDA, netcat:TP06R
- removed TP26: MSCL, netcat:TP06R
- removed TP5: TSDA, netcat:TP06R
- added IC26: DS18B20U, netcat:USOP-8
- added R10, R11: 4.7k, netcat:R0402
- added SJ2, SJ3: (no value), netcat:SJ2
- IC14: device netcat:SO-08 -> netcat:UDFN8-3X2
- OSC2: value 8 mhz -> 8 MHz
- OSC3: value 32.768k -> 32.768 KHz
- R13, R38, R39, R8: value 10k -> 4.7k
- R15: value 1M -> 300k
- moved C43 3.47 mm to (85.8, 47.2), turned to 0 degrees
- moved C54 2.77 mm to (65.3, 34.1), turned to 0 degrees
- moved IC14 2.19 mm to (83.2, 45.5), turned to 270 degrees
- moved R5 1.45 mm to (11.9, 38.4), turned to 270 degrees
- moved R49 1.35 mm to (100.4, 52.2)
- moved C66 1.25 mm to (100.4, 51.1)
- moved OSC4 1.20 mm to (64.7, 32.0)
- moved Q10 0.63 mm to (108.0, 24.3), turned to 180 degrees
- moved C6 0.56 mm to (50.9, 37.2)
- moved R45 0.56 mm to (50.9, 36.0)
- moved R16 0.51 mm to (50.9, 34.7)
- moved R36 0.40 mm to (59.4, 37.5)
- moved LED2 0.40 mm to (59.4, 40.0)
- moved R23 0.35 mm to (100.4, 50.0)
- moved Q2 0.30 mm to (60.9, 35.5)
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Connections:
- new net 1W: IC1.23, IC26.4
- net 3.3V: now also IC26.3, R10.1, R11.1
- net EE_I2C_SCL: now also SJ3.1; no longer TP26.TP
- net EE_I2C_SDA: now also SJ2.1; no longer TP25.TP
- net GND: now also IC26.5
- net TS_SCL: now also R10.2, SJ3.2; no longer TP13.TP
- net TS_SDA: now also R11.2, SJ2.2; no longer TP5.TP
Routing:
- net 1W: track 0.00 -> 50.3 mm, vias 0 -> 2
- net TS_SDA: track 52.5 -> 59.2 mm
- net TS_SCL: track 55.0 -> 60.3 mm
- net 3.3V: track 781.8 -> 776.7 mm, vias 50 -> 48
- net GND: track 37.3 -> 42.1 mm, vias 439 -> 436
- net EE_I2C_SDA: track 156.0 -> 158.3 mm
- net V_USB: track 31.9 -> 33.8 mm
- net LED_ST_EN: track 35.8 -> 37.5 mm
- net BAT_SENS: track 57.1 -> 58.3 mm
- net EE_I2C_SCL: track 161.5 -> 160.4 mm
- net GSM_NL: track 7.58 -> 6.56 mm
- net BUT2: track 47.7 -> 48.7 mm
- net SDHC_ST: track 42.4 -> 41.4 mm
- net N$69: track 10.6 -> 9.68 mm
- net PWR_SHDN: track 60.8 -> 61.6 mm
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
Commit message: new battery connection mechanism
Parts:
- removed X2: BAT, netcat:1X03
- U$3: value GALAXY_S3MINI_BATTARY -> GALAXY_BATTARY_S4; device netcat:GALAXY_S3MINI_BATTARY -> netcat:GALAXY_S4_BATTARY
- moved R14 6.59 mm to (5.00, 41.4), turned to 0 degrees
- moved IC20 6.50 mm to (2.45, 48.0), turned to 90 degrees
- moved C61 5.71 mm to (7.20, 50.8), turned to 0 degrees
- moved TP20 5.11 mm to (13.9, 57.2)
- moved C2 3.87 mm to (11.5, 43.2), turned to 0 degrees
- moved R15 2.72 mm to (2.20, 41.4), turned to 0 degrees
- moved R37 2.71 mm to (5.00, 43.2)
- moved LED3 2.67 mm to (2.20, 43.2)
- moved TP22 1.35 mm to (16.6, 57.2)
- moved U$3 0.71 mm to (40.5, 32.0)
- moved R6 0.65 mm to (8.90, 57.2)
- moved SW2 0.25 mm to (13.4, 62.5)
Connections:
- net GND: no longer X2.3
- net V_BAT: no longer X2.1
Routing:
- net DMIC_DAT: track 145.4 -> 151.2 mm
- net V_BAT: track 71.2 -> 65.8 mm, vias 2 -> 3
- net BAT_SENS: track 58.3 -> 52.9 mm
- net DMIC_CLK: track 145.6 -> 149.4 mm
- net 3.3V: track 776.7 -> 773.2 mm
- net GND: track 42.1 -> 44.8 mm, vias 436 -> 435
- net RINGP: track 172.7 -> 170.0 mm
- net RINGN: track 186.3 -> 184.5 mm
- net PWR_OTG_MODE: track 46.0 -> 47.7 mm
- net PWR_BUT: track 206.9 -> 205.6 mm
- net GPIO_FPGA1: track 117.3 -> 116.4 mm
- net BAT_CHG: track 50.3 -> 49.4 mm
- net V_SYS: track 24.0 -> 23.4 mm
