File: redphone.brd (EAGLE design)
At the start: 156 x 65 mm, 239 parts, among them IC1 EP4CE6E22, IC10 MPU9250, IC11 PCA9633TK, IC13 TPS63000, IC14 24LC256, IC16 EPCS4SI8N, IC18 WM8903, IC19 AT25SF041, IC2 STM32F429ZIT, IC20 MP34DT01, IC21 PT4181, IC22 MAX8903A, IC23 NRF24L01+, IC24 BME280, IC25 APDS-9960, IC26 DS18B20U, IC27 MC-1010-G, IC28 MAX2659, IC3 MT48LC16M16A2TG, IC4 MAX8815A, IC5 LP3990TL, IC6 LP3990TL, IC7 TPS63001, IC8 ESP8266, IC9 SIM800C, Q1 IRLML2502, Q2 NTA4153NT1G, Q3 BCR133W, Q4 NTA4153NT1G, Q5 NTA4153NT1G, Q6 IRLML2502, Q7 16MHz, Q8 NTA4153NT1G, SW1 PWR, SW2 CAM, SW3 VOL+, SW4 VOL-, X1 MICRO_SIM_SDS, X10 AUDIO-JACKSMD, X13 OV2640, X14 UFL, X18 FPC_I9500_BAT_CON, X3 RM68120_LCD, X5 LG_P715_TS, Y1 2.4Ghz, Y3 2.4Ghz, Y4 GSM_PCB, Y5 2.4Ghz

Commit message: label upd, added more tps, route fix, dfc fix, round corners
Parts:
- removed U$3: GALAXY_BATTARY_S4, netcat:GALAXY_S4_BATTARY
- added BATTARY_PLACE: GALAXY_BATTARY_S4, netcat:GALAXY_BATTARY_S4
- added C11: 4.7p, netcat:R0603
- added IC12: HDC1000, netcat:DSBGA8
- added IO: IO, netcat:TP06R
- added R31: 100, netcat:R0402
- added SCL10, TP28, TP31, TP32: RX, netcat:TP06R
- added SCL11, SCL7, TP29, TP30: TX, netcat:TP06R
- added SCL4: PC1, netcat:TP06R
- added SCL5: RST, netcat:TP06R
- added SCL6: TS_INT, netcat:TP06R
- added SCL8: CLK, netcat:TP06R
- added SCL9: PA15, netcat:TP06R
- added SJ4: (no value), netcat:SJ2
- added TP20: V_USB, netcat:TP06R
- added TP25: CC2, netcat:TP06R
- added TP26: NL, netcat:TP06R
- added TP27: PK, netcat:TP06R
- added TP33, TP34, TP35, TP36, TP37, TP38: GND, netcat:TP06R
- added TP39: TMS, netcat:TP06R
- added TP40: TCK, netcat:TP06R
- added TP41: TDO, netcat:TP06R
- added TP42: TDI, netcat:TP06R
- added X7: (no value), netcat:PLS2-1X01
- C7: value 100u -> 10u
- IC23: value NRF24L01+ -> NRF24L01
- TP1: value TP -> IO124
- TP10: value DONE -> CD
- TP11: value MISO -> MOSI
- TP12: value MOSI -> MISO
- TP13: value 3 -> 4
- TP2: value TP -> IO129
- TP24: value TSI -> VBAT
- TP9: value 1 -> 2
- X16: value (none) -> USB
- moved TP24 81.3 mm to (-4.50, 52.0)
- moved C43 41.7 mm to (104.8, 10.1)
- moved R39 22.3 mm to (86.5, 44.5), turned to 90 degrees
- moved R38 17.6 mm to (88.4, 41.1), turned to 270 degrees
- moved TP13 9.20 mm to (-4.50, 44.5)
- moved TP9 9.20 mm to (-4.50, 49.5)
- moved X18 9.00 mm to (-5.00, 54.8)
- moved C46 7.13 mm to (93.5, 10.0)
- moved B2 4.70 mm to (128.3, 39.0)
- moved IC11 4.05 mm to (122.5, 12.6)
- moved IC25 4.00 mm to (123.0, 54.0)
- moved LED1 4.00 mm to (123.0, 17.0)
- moved R6 4.00 mm to (124.8, 19.0)
- moved R7 4.00 mm to (124.5, 16.3)
- moved R9 4.00 mm to (123.0, 19.8)
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Connections:
- net LED_ST_EN renamed IO124
- net NAV_INT1 renamed IO129
- removed net SIM_DET: IC9.14
- new net N$106: IC2.27, SCL4.TP
- new net N$107: IC2.110, SCL9.TP
- new net N$108: IC26.3, SJ4.2
- new net N$109: C11.2, IC9.28
- net 3.3V: now also IC12.B1, SJ4.1; no longer IC26.3
- net BL_RST: now also SCL5.TP
- net FPGA_RX: now also TP32.TP
- net FPGA_TX: now also SCL7.TP
- net GND: now also C11.1, IC12.B2, IC12.C1, IC12.D1, TP33.TP, TP34.TP, TP35.TP, TP36.TP, TP37.TP, X7.1
- net GND_BAT: now also TP38.TP, X18.3; no longer X18.4
- net GPS_RX: now also TP31.TP
- net GPS_TX: now also TP30.TP
- net GSM_NL: now also TP26.TP
- net GSM_RX: now also TP28.TP
- net GSM_TX: now also TP29.TP
- net JTAG_TCK: now also TP40.TP
- net JTAG_TDI: now also TP42.TP
- net JTAG_TDO: now also TP41.TP
- net JTAG_TMS: now also TP39.TP
- net N$104: now also X18.2; no longer X18.1
- net N$105: now also X18.4; no longer X18.3
- net N$15: now also VD4.A; no longer VD4.C
- net N$69: now also TP27.TP
- net N$9: now also R31.1
- net NAV_I2C_SCL: now also IC12.A1
- net NAV_I2C_SDA: now also IC12.A2
- net PWR_BUT: now also VD4.C; no longer VD4.A
- net SWD_CLK: now also SCL8.TP
- net SWD_IO: now also IO.TP
- net TS_INT: now also SCL6.TP; no longer TP24.TP
- net UART_EXT_RX: now also SCL10.TP
- net UART_EXT_TX: now also SCL11.TP
- net USB_CC2: now also TP25.TP
- net V_BAT2: now also TP24.TP, X18.1; no longer X18.2
- net V_INT: now also R31.2
- net V_USB: now also TP20.TP
Routing:
- net 3.3V: track 776.2 -> 792.5 mm, vias 49 -> 48
- net GND: track 54.6 -> 45.0 mm, vias 499 -> 528
- net N$59: track 14.4 -> 6.84 mm
- net V_INT: track 62.7 -> 67.8 mm
- net V_BAT2: track 12.1 -> 16.4 mm
- net N$108: track 0.00 -> 4.12 mm
- net NAV_I2C_SDA: track 53.3 -> 57.3 mm, vias 4 -> 5
- net NAV_I2C_SCL: track 55.2 -> 59.1 mm, vias 3 -> 4
- net V_USB: track 31.9 -> 34.6 mm, vias 1 -> 2
- net SDIO_CLK: track 49.8 -> 47.2 mm
- net N$107: track 0.00 -> 2.57 mm
- net JTAG_TMS: track 101.1 -> 103.5 mm
- net DMIC_CLK: track 147.0 -> 149.3 mm
- net SD_SI: track 12.2 -> 9.96 mm, vias 2 -> 0
- net DMIC_DAT: track 148.5 -> 150.8 mm
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Other:
- board size 156 x 65 mm -> 145 x 65 mm
- board text added: "redphone v1.1"
- board text removed: "geeksphone v1.0"

Commit message: fix MPU9250 pkg
Parts:
- IC10: device netcat:QFN24-EP -> netcat:QFN24-3X3
- SJ1: value SJ3 -> (none)
- moved C26 0.21 mm to (113.2, 9.95)
Routing:
- net GND: track 45.0 -> 48.2 mm
- net 3.3V: track 792.5 -> 795.0 mm
- net NAV_INT0: track 40.3 -> 41.1 mm
- net N$78: track 1.83 -> 2.54 mm
- net NAV_I2C_SDA: track 57.3 -> 57.8 mm
- net NAV_I2C_SCL: track 59.1 -> 59.6 mm

Commit message: route & schematic fix, connect PWR_BUT to fpga, new IO89 tp
Parts:
- TP2: value IO129 -> IO89
- moved TP2 19.6 mm to (67.8, 4.65)
- moved R3 1.12 mm to (70.2, 4.65)
- moved TP5 0.46 mm to (66.7, 5.40)
- moved L6 0.25 mm to (106.2, 54.9)
- moved TP10 0.22 mm to (68.7, 4.65)
Connections:
- net BQ0 renamed SDR_BQ0
- net BQ1 renamed SDR_BQ1
- removed net IO129: IC1.129, TP2.TP
- new net N$110: IC1.89, TP2.TP
- net PWR_BUT: now also IC1.129
Routing:
- net PWR_BUT: track 188.9 -> 217.1 mm, vias 9 -> 10
- net 3.3V: track 795.0 -> 787.8 mm, vias 48 -> 49
- net N$110: track 0.00 -> 2.85 mm
- net GND: track 48.2 -> 50.1 mm, vias 528 -> 532
- net IO129: track 1.92 -> 0.00 mm
- net FPGA_IO3: track 16.9 -> 15.8 mm
- net N$4: track 2.86 -> 3.70 mm
- net 2.5V: track 136.2 -> 137.0 mm

Commit message: fix dimension, silk, mdl connectors, added extra tps & led on 3.3v
Parts:
- removed X11, X12, X17, X2, X4, X6, X7, X8, X9: (no value), netcat:PLS2-1X01
- added R50: 330, netcat:R0402
- added TP43, TP44: 3.3v, netcat:TP06R
- added TP45, TP46, TP47, TP48, TP49, TP50, TP51, TP52, TP53, TP54, TP55, TP56, TP57, TP58, TP59, TP60, TP61, TP62, TP63, TP64, TP65, TP66, TP67, TP68, TP69, TP70, TP71, TP72, TP73, TP74, TP75, TP76, TP77, TP78, TP79, TP80, TP81, TP82: (no value), netcat:TP065RH
- added TP83: OTG, netcat:TP06R
- added TP84: SHDN, netcat:TP06R
- added VD9: (no value), netcat:LED0603
- Q1, Q6: value IRLML2502 -> IRLML6402
- Q3: device netcat:SOT323 -> netcat:SOT23
- TP20: value V_USB -> VUSB
- moved R12 1.35 mm to (12.6, 40.5), turned to 0 degrees
- moved R37 1.20 mm to (5.20, 41.4)
- moved R6 1.12 mm to (125.8, 19.5)
- moved R9 1.12 mm to (124.0, 20.2)
- moved B2 1.00 mm to (129.3, 39.0)
- moved IC11 1.00 mm to (123.5, 12.6)
- moved VD6 0.99 mm to (1.90, 41.4), turned to 90 degrees
- moved R7 0.71 mm to (125.0, 16.8)
- moved VD4 0.51 mm to (12.4, 53.2)
- moved LED1 0.50 mm to (123.0, 17.5)
- moved Q3 0.25 mm to (15.1, 53.6)
Connections:
- new net N$23: R50.1, VD9.A
- net 3.3V: now also R50.2, TP43.TP, TP44.TP, TP45.1, TP68.1; no longer X2.1
- net 3.3V2: now also TP79.1
- net FPGA_IO0: now also TP48.1; no longer X9.1
- net FPGA_IO1: now also TP46.1; no longer X11.1
- net FPGA_IO2: now also TP47.1; no longer X4.1
- net FPGA_IO3: now also TP49.1; no longer X6.1
- net GND: now also TP50.1, TP51.1, TP52.1, TP53.1, TP54.1, TP55.1, TP56.1, TP57.1, TP59.1, TP60.1, TP61.1, TP65.1, VD9.C; no longer X12.1, X17.1, X7.1, X8.1
- net GND2: now also TP76.1
- net GND_BAT: now also TP70.1, TP71.1, TP72.1
- net NAV_I2C_SCL: now also TP67.1
- net NAV_I2C_SCL2: now also TP78.1
- net NAV_I2C_SDA: now also TP66.1
- net NAV_I2C_SDA2: now also TP77.1
- net PWR_OTG_MODE: now also TP83.TP
- net PWR_SHDN: now also TP84.TP
- net SPKRN: now also TP64.1
- net SPKRN2: now also TP80.1
- net SPKRP: now also TP63.1
- net SPKRP2: now also TP81.1
- net V_BAT: now also TP58.1
- net V_BAT2: now also TP69.1
Routing:
- net 3.3V: track 787.8 -> 794.1 mm, vias 49 -> 48
- net N$80: track 4.35 -> 1.90 mm
- net N$23: track 0.00 -> 1.90 mm, vias 1 -> 0
- net 3.3V2: track 57.0 -> 58.9 mm, vias 1 -> 3
- net GND: track 50.1 -> 51.9 mm, vias 532 -> 523
- net PWR_OTG_MODE: track 47.0 -> 48.4 mm
- net PWR_SHDN: track 64.4 -> 65.7 mm
- net V_USB: track 34.6 -> 35.8 mm
- net N$40: track 1.52 -> 2.52 mm
- net GND2: track 50.0 -> 51.0 mm, vias 3 -> 2
- net N$76: track 6.15 -> 7.04 mm
- net N$79: track 11.2 -> 11.7 mm
- net N$41: track 1.17 -> 1.67 mm
- net NAV_I2C_SCL2: track 54.8 -> 55.2 mm, vias 2 -> 1
- net NAV_I2C_SDA2: track 57.4 -> 57.8 mm, vias 2 -> 1
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Other:
- board size 145 x 65 mm -> 146 x 65 mm

Commit message: fix pkg of gps lna, cap & res values fix, drc fix
Parts:
- C10: value (none) -> 470p
- L3: value (none) -> 6.8uH
- R46: value 1M -> 1.5M
- R51: value 220k -> 215k
- moved IC28 0.35 mm to (21.1, 56.3)
Routing:
- net N$72: track 1.25 -> 1.95 mm

Commit message: swap EPCS pins, added res
Parts:
- added R52, R56, R58: 10k, netcat:R0402
- IC16: value EPCS4SI8N -> EPCS16N
- moved C68 2.04 mm to (89.0, 43.0), turned to 0 degrees
- moved R38 2.04 mm to (89.0, 39.2), turned to 180 degrees
Connections:
- net 3.3V: now also R52.1, R56.1, R58.1
- net EPCS_!CS: now also IC16.1, R56.2; no longer IC16.5
- net EPCS_ASDI: now also IC16.5, R58.2; no longer IC16.1
- net EPCS_DATA: now also R52.2
Routing:
- net EPCS_!CS: track 16.1 -> 26.6 mm
- net EPCS_ASDI: track 23.0 -> 17.9 mm
- net EPCS_DATA: track 24.2 -> 28.6 mm
- net 3.3V: track 794.1 -> 796.3 mm
- net EE_I2C_SDA: track 139.7 -> 138.4 mm

Commit message: connect lcd dc-dc to V_INT, connect AQ13 to FPGA
Parts:
- added R59: 330, netcat:R0402
- added SCL12: PC1, netcat:TP06R
- added TP85: PPS, netcat:TP06R
- added VD10: (no value), netcat:LED0603
- TP15: value VINT -> V_INT
- moved TP43 3.61 mm to (105.7, 26.9)
- moved TP1 0.30 mm to (105.7, 24.9)
- moved TP34 0.30 mm to (105.7, 25.9)
- moved R50 0.15 mm to (5.20, 43.0)
- moved VD9 0.15 mm to (1.90, 43.0)
Connections:
- new net N$25: IC2.7, SCL12.TP
- new net N$77: R59.1, VD10.A
- new net N$88: IC27.4, TP85.TP
- net 3.3V: no longer IC21.6, L10.1
- net AQ13: now also IC1.25
- net GND: now also VD10.C
- net IO124: now also R59.2
- net V_INT: now also IC21.6, L10.1
Routing:
- net V_INT: track 67.7 -> 241.3 mm, vias 0 -> 2
- net 3.3V: track 796.3 -> 792.0 mm, vias 48 -> 47
- net N$25: track 0.00 -> 2.53 mm
- net AQ13: track 87.1 -> 89.4 mm, vias 2 -> 3
- net N$77: track 0.00 -> 2.00 mm
- net EE_I2C_SDA: track 138.4 -> 140.1 mm
- net N$88: track 0.00 -> 1.65 mm
- net IO124: track 32.4 -> 33.4 mm
- net 2.5V: track 137.0 -> 137.7 mm
- net DQ3: track 94.3 -> 95.0 mm
- net SPKRN: track 31.2 -> 30.6 mm
- net SPKRP: track 27.7 -> 27.1 mm
- net PWR_BUT: track 217.3 -> 217.7 mm, vias 10 -> 8

Commit message: start rerouting
Parts:
- removed C1, C2, C28, C29, C5, C69, C7: 10u, netcat:SMC_A
- removed C10: 470p, netcat:R0402
- removed C18, C3, C4, C43, C6, C66, C72, C79: 100n, netcat:R0402
- removed C21, C22: 22p, netcat:R0402
- removed C23: 33n, netcat:R0402
- removed C24: 2.2n, netcat:R0402
- removed C25: 4.7p, netcat:R0402
- removed C27: 1.5p, netcat:R0402
- removed C70: 220n, netcat:R0402
- removed C9: 100p, netcat:R0402
- removed IC12: HDC1000, netcat:DSBGA8
- removed IC13: TPS63000, netcat:DFN10-3X3
- removed IC14: 24LC256, netcat:UDFN8-3X2
- removed IC21: PT4181, netcat:SOT23-6
- removed IC22: MAX8903A, netcat:TQFN28-EP
- removed IC23: NRF24L01, netcat:QFN20
- removed IC26: DS18B20U, netcat:USOP-8
- removed IC27: MC-1010-G, netcat:MC-1010-G
- removed IC28: MAX2659, netcat:UDFN6
- removed IC5, IC6: LP3990TL, netcat:DSBGA
- removed IC7: TPS63001, netcat:DFN10-3X3
- removed IO: IO, netcat:TP06R
- removed L1, L2, L7: 2.2uH, netcat:CDRH2D18LD
- removed L10: 22uH, netcat:L3216C
- removed L3: 6.8uH, netcat:R0402
- removed L4: 2.7nH, netcat:R0402
- removed L5: 8.2nH, netcat:R0402
- removed L8: 3.9nH, netcat:R0402
- removed LED2, VD10, VD6, VD7, VD8, VD9: (no value), netcat:LED0603
- removed Q1, Q6: IRLML6402, netcat:SOT23
- removed Q2, Q5, Q8: NTA4153NT1G, netcat:SOT-416
- removed Q3: BCR133W, netcat:SOT23
- removed Q7: 16MHz, netcat:3225
- removed R10, R11, R13, R38, R39, R8: 4.7k, netcat:R0402
- removed R12, R14, R16, R19, R35, R4, R43, R5, R57: 100k, netcat:R0402
- removed R15: 300k, netcat:R0402
- removed R22: 1.5k, netcat:R0402
- removed R24: 1M, netcat:R0402
- removed R25: 22k, netcat:R0402
- removed R31, R45: 100, netcat:R0402
- removed R34: 3k, netcat:R0402
- removed R36, R37, R50, R59: 330, netcat:R0402
- removed R46: 1.5M, netcat:R0402
- removed R47: 5.2, netcat:R0402
- removed R51: 215k, netcat:R0402
- removed R52, R56, R58: 10k, netcat:R0402
- removed SCL, TP8: SCL, netcat:TP06R
- removed SCL1: PB2, netcat:TP06R
- removed SCL10, TP31, TP32: RX, netcat:TP06R
- removed SCL11, SCL7, TP30: TX, netcat:TP06R
- removed SCL12, SCL4: PC1, netcat:TP06R
- removed SCL2: PA4, netcat:TP06R
- removed SCL3: PB0, netcat:TP06R
- removed SCL8, TP18: CLK, netcat:TP06R
- removed SCL9: PA15, netcat:TP06R
- removed SJ1: (no value), netcat:SJ3
- removed SJ2, SJ3, SJ4: (no value), netcat:SJ2
- removed TP1: IO124, netcat:TP06R
- removed TP10: CD, netcat:TP06R
- removed TP11: MOSI, netcat:TP06R
- removed TP12: MISO, netcat:TP06R
- removed TP14: 5v, netcat:TP06R
- removed TP15: V_INT, netcat:TP06R
- removed TP16: 2.5v, netcat:TP06R
- removed TP17: 1.2v, netcat:TP06R
- removed TP19, TP43, TP44: 3.3v, netcat:TP06R
- removed TP2: IO89, netcat:TP06R
- removed TP20: VUSB, netcat:TP06R
- removed TP22: 4v, netcat:TP06R
- removed TP25: CC2, netcat:TP06R
- removed TP33, TP34, TP35, TP36, TP37: GND, netcat:TP06R
- removed TP39: TMS, netcat:TP06R
- removed TP40: TCK, netcat:TP06R
- removed TP41: TDO, netcat:TP06R
- removed TP42: TDI, netcat:TP06R
- removed TP45, TP46, TP47, TP48, TP49, TP50, TP51, TP52, TP53: (no value), netcat:TP065RH
- removed TP5: IO88, netcat:TP06R
- removed TP7: SDA, netcat:TP06R
- removed TP83: OTG, netcat:TP06R
- removed TP84: SHDN, netcat:TP06R
- removed TP85: PPS, netcat:TP06R
- removed VD1, VD3: STPS0520Z, netcat:SOD123
- removed VD4: (no value), netcat:SOD523
- removed X13: OV2640, netcat:MOLEX-52437-2491
- removed X14: UFL, netcat:UFL-R-SMT
- removed Y2: (no value), netcat:ANTENNA_CHIP_2X9
- removed Y3: 2.4Ghz, netcat:ANTENNA_CHIP_2X5
- IC3: value MT48LC16M16A2TG -> MT48LC16M16A2B4; device netcat:TSOPII-54 -> netcat:VFBGA-54
- IC4: value MAX8815A -> MT48LC16M16A2B4; device netcat:DFN10-3X3 -> netcat:VFBGA-54
- moved IC4 36.6 mm to (45.4, 12.5), turned to 0 degrees
- moved SCL5 31.5 mm to (25.9, 5.53)
- moved TP21 19.4 mm to (94.8, 16.4)
- moved R30 14.0 mm to (91.5, 13.3), turned to 90 degrees
- moved TP23 13.8 mm to (94.2, 26.4)
- moved C39 12.8 mm to (92.7, 13.3), turned to 90 degrees
- moved C55 12.0 mm to (40.6, 5.18), turned to 0 degrees
- moved C63 9.14 mm to (26.4, 31.4), turned to 0 degrees
- moved C45 8.92 mm to (90.1, 13.4), turned to 90 degrees
- moved Q4 8.65 mm to (59.0, 43.3)
- moved C49 8.52 mm to (90.8, 24.5), turned to 90 degrees
- moved C51 7.21 mm to (94.2, 24.5), turned to 270 degrees
- moved R41 6.85 mm to (95.8, 24.7), turned to 90 degrees
- moved IC3 6.84 mm to (45.4, 24.4), turned to 0 degrees
- moved R48 6.52 mm to (106.0, 9.72), turned to 90 degrees
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Connections:
- removed net !LCD_BL_EN: IC1.106, IC21.4, R43.2
- removed net 1W: IC1.23, IC26.4
- removed net ANT: C27.2, Y3.FEED
- removed net FPGA_IO0: IC1.104, TP48.1
- removed net FPGA_IO1: IC1.105, TP46.1
- removed net FPGA_IO2: IC1.90, TP47.1
- removed net FPGA_IO3: IC1.91, TP49.1
- removed net GPIO_FPGA0: IC1.120, X16.A8
- removed net GPIO_FPGA1: IC1.121, X16.B8
- removed net IO124: IC1.124, R59.2, TP1.TP
- removed net N$1: IC4.10, IC4.6, IC4.7, IC4.9, Q6.3, TP14.TP
- removed net N$10: C6.1, IC13.7, IC13.8, R45.1
- removed net N$106: IC2.27, SCL4.TP
- removed net N$107: IC2.110, SCL9.TP
- removed net N$108: IC26.3, SJ4.2
- removed net N$11: IC7.4, L2.1
- removed net N$110: IC1.89, TP2.TP
- removed net N$13: IC4.3, L1.2, VD1.C
- removed net N$14: IC7.2, L2.2
- removed net N$15: Q1.1, Q3.3, R4.1, VD4.A
- removed net N$18: Q2.3, R36.1
- removed net N$19: IC13.10, R46.2, R51.1
- removed net N$20: IC13.4, L7.1
- removed net N$21: C10.1, Y2.FEED
- removed net N$23: R50.1, VD9.A
- removed net N$25: IC2.7, SCL12.TP
- removed net N$28: IC13.2, L7.2
- removed net N$30: C21.1, IC23.9, Q7.3, R24.1
- removed net N$31: C22.1, IC23.10, Q7.1, R24.2
- removed net N$32: IC23.13, L5.2, L8.1
- removed net N$33: C24.1, C25.1, IC23.11, L4.2
- removed net N$34: IC23.16, R25.1
- removed net N$35: C23.1, IC23.19
- removed net N$36: IC23.12, L4.1, L5.1
- removed net N$37: C27.1, L8.2
- removed net N$5: Q6.1, Q8.3, R5.2
- removed net N$6: C72.2, IC22.5, IC22.7, IC22.9
- removed net N$61: C10.2, L3.1
- removed net N$65: IC22.11, R34.2
- removed net N$66: IC22.13, R22.2
- removed net N$67: LED2.C, R36.2
- removed net N$7: IC1.88, TP5.TP
- removed net N$72: IC28.3, L3.2
- removed net N$73: Q5.3, VD7.C, VD8.C
- removed net N$74: IC2.40, SCL2.TP
- removed net N$75: IC2.48, SCL1.TP
- removed net N$77: R59.1, VD10.A
- removed net N$8: IC4.1, IC4.2, L1.1
- removed net N$80: R37.1, VD6.A
- removed net N$84: IC21.1, L10.2, VD3.A
- removed net N$88: IC27.4, TP85.TP
- removed net N$89: SJ1.3, X14.SIG
- removed net N$9: C79.1, IC7.6, IC7.7, IC7.8, R31.1
- removed net N$90: SJ1.1, Y4.S
- removed net N$93: R19.1, X13.6
- removed net N$97: IC2.46, SCL3.TP
- removed net N$99: IC22.14, R57.1
- removed net OV_CLK: IC1.144, TP18.TP, X13.13
- removed net OV_D0: IC1.137, X13.19
- removed net OV_D1: IC1.135, X13.21
- removed net OV_D2: IC1.133, X13.22
- removed net OV_D3: IC1.136, X13.20
- removed net OV_D4: IC1.138, X13.18
- removed net OV_D5: IC1.142, X13.16
- removed net OV_D6: IC1.143, X13.14
- removed net OV_D7: IC1.1, X13.12
- removed net OV_HSYNC: IC1.2, X13.9
- removed net OV_PCLK: IC1.141, X13.17
- removed net OV_VSYNC: IC1.3, X13.7
- removed net RF_OUT: IC27.11, IC28.6
- removed net VCC_RF: C9.1, IC27.14, IC28.4, IC28.5
- removed net V_INT: C7.+, IC13.5, IC21.6, IC5.B2, IC6.B2, IC7.5, L10.1, Q1.3, R31.2, R45.2, TP15.TP
- removed net V_SYS: IC22.23, IC22.24, Q1.2, R4.2
- removed net V_USB: C2.+, IC22.17, Q6.2, R37.2, R5.1, TP20.TP, X16.A4, X16.A9, X16.B4, X16.B9
- net !GSM_EN: no longer IC13.6, R16.2
- net !NRF_CS: no longer IC23.2
- net 1.2V: no longer C28.+, C4.1, IC6.B1, TP17.TP, X13.10
- net 2.5V: no longer C29.+, C3.1, IC5.B1, TP16.TP, X13.11, X13.4
- net 3.3V: now also IC3.A7, IC3.A9, IC3.B3, IC3.C7, IC3.D3, IC3.E7, IC3.J9; no longer C1.+, C18.1, C43.2, C66.1, C69.+, IC12.B1, IC14.8, IC23.15, IC23.18, IC23.7, IC27.6, IC27.8, IC3.1, IC3.14, IC3.27, IC3.3, IC3.43, IC3.49, IC3.9, IC7.1, IC7.10, LED2.A, R10.1, R11.1, R13.1, R19.2, R35.1, R38.1, R39.1, R50.2, R52.1, R56.1, R58.1, R8.1, SJ4.1, TP19.TP, TP43.TP, TP44.TP, TP45.1, VD1.A, VD7.A, VD8.A
- net 4.0V: no longer C5.+, IC13.1, R46.1, TP22.TP
- net AQ0: now also IC3.H7; no longer IC1.77, IC3.23
- net AQ1: now also IC3.H8; no longer IC1.80, IC3.24
- net AQ10: now also IC3.H9; no longer IC1.76, IC3.22
- net AQ11: now also IC3.G2; no longer IC1.66, IC3.35
- net AQ12: now also IC3.G1; no longer IC1.65, IC3.36
- net AQ13: no longer IC1.25, X3.42
- net AQ2: now also IC3.J8; no longer IC1.83, IC3.25
- net AQ3: now also IC3.J7; no longer IC1.84, IC3.26
- net AQ4: now also IC3.J3; no longer IC1.72, IC3.29
- net AQ5: now also IC3.J2; no longer IC1.71, IC3.30
- net AQ6: now also IC3.H3; no longer IC1.70, IC3.31
- net AQ7: now also IC3.H2; no longer IC1.69, IC3.32
- net AQ8: now also IC3.H1; no longer IC1.68, IC3.33
- net AQ9: now also IC3.G3; no longer IC1.67, IC3.34
- net AUDIO_INT: no longer IC1.114
- net BAT_CHG: no longer IC22.22, R35.2
- net BAT_SENS: no longer R14.1, R15.2
- net BL_RST: no longer X16.A5
- net DQ0: now also IC3.A8; no longer IC1.30, IC3.2, X3.11
- net DQ1: now also IC3.B9; no longer IC1.28, IC3.4, X3.12
- net DQ10: now also IC3.D1; no longer IC1.54, IC3.45, X3.21
- net DQ11: now also IC3.C2; no longer IC1.53, IC3.47, X3.22
- net DQ12: now also IC3.C1; no longer IC1.52, IC3.48, X3.23
- net DQ13: now also IC3.B2; no longer IC1.51, IC3.50, X3.24
- net DQ14: now also IC3.B1; no longer IC1.50, IC3.51, X3.25
- net DQ15: now also IC3.A2; no longer IC1.49, IC3.53, X3.26
- net DQ2: now also IC3.B8; no longer IC1.32, IC3.5, X3.13
- net DQ3: now also IC3.C9; no longer IC1.31, IC3.7, X3.14
- net DQ4: now also IC3.C8; no longer IC1.33, IC3.8, X3.15
- net DQ5: now also IC3.D9; no longer IC1.34, IC3.10, X3.16
- net DQ6: now also IC3.D8; no longer IC1.38, IC3.11, X3.17
- net DQ7: now also IC3.E9; no longer IC1.39, IC3.13, X3.18
- net DQ8: now also IC3.E1; no longer IC1.58, IC3.42, X3.19
- net DQ9: now also IC3.D2; no longer IC1.55, IC3.44, X3.20
- net EE_I2C_SCL: no longer IC1.126, IC14.6, R39.2, SJ3.1, TP8.TP, X13.5
- net EE_I2C_SDA: no longer IC1.125, IC14.5, R38.2, SJ2.1, TP7.TP, X13.3
- net EPCS_!CS: no longer IC1.8, R56.2
- net EPCS_ASDI: no longer IC1.6, R58.2
- net EPCS_DATA: no longer IC1.13, R52.2
- net FMC_!E1: no longer IC1.100, X3.39
- net FMC_!E2: no longer IC1.119
- net FMC_!OE: no longer IC1.103, X3.40
- net FMC_!WE: no longer IC1.101, X3.41
- net FPGA_EN: no longer IC5.A2, IC6.A2
- net FPGA_MISO: no longer IC1.86, TP12.TP
- net FPGA_MOSI: no longer IC1.85, TP11.TP
- net FPGA_RX: no longer IC1.99, TP32.TP
- net FPGA_SCL: no longer IC1.87, SCL.TP
- net FPGA_TX: no longer IC1.98, SCL7.TP
- net GND: now also IC3.A1, IC3.A3, IC3.B7, IC3.C3, IC3.D7, IC3.E3, IC3.J1; no longer C1.-, C18.2, C2.-, C21.2, C22.2, C23.2, C24.2, C25.2, C28.-, C29.-, C3.2, C4.2, C43.1, C5.-, C6.2, C66.2, C69.-, C7.-, C70.2, C72.1, C79.2, C9.2, IC12.B2, IC12.C1, IC12.D1, IC13.3, IC13.9, IC13.PPAD, IC14.1, IC14.2, IC14.3, IC14.4, IC14.7, IC21.2, IC22.1, IC22.10, IC22.12, IC22.16, IC22.2, IC22.3, IC22.4, IC22.EP, IC23.0, IC23.14, IC23.17, IC23.20, IC23.8, IC26.5, IC27.1, IC27.10, IC27.12, IC28.1, IC28.2, IC3.12, IC3.28, IC3.41, IC3.46, IC3.52, IC3.54, IC3.6, IC4.5, IC4.8, IC4.PPAD, IC5.A1, IC6.A1, IC7.3, IC7.9, IC7.PPAD, Q2.2, Q3.2, Q5.2, Q7.2, Q7.4, Q8.2, R12.1, R15.1, R16.1, R22.1, R25.2, R34.1, R43.1, R47.1, R51.2, R57.2, TP33.TP, TP34.TP, TP35.TP, TP36.TP, TP37.TP, TP50.1, TP51.1, TP52.1, TP53.1, VD10.C, VD6.C, VD9.C, X13.15, X13.2, X14.GND@0, X14.GND@1
- net GPS_RX: no longer IC27.3, TP31.TP
- net GPS_TX: no longer IC27.2, TP30.TP
- net GSM_ANT: now also Y4.S; no longer SJ1.2
- net GSM_NL: no longer Q2.1
- net JTAG_TCK: no longer TP40.TP, X16.B11
- net JTAG_TDI: no longer TP42.TP, X16.A10
- net JTAG_TDO: no longer TP41.TP, X16.B2
- net JTAG_TMS: no longer TP39.TP, X16.B10
- net LCD_BL_GND: no longer IC21.3, R47.2
- net LCD_BL_PWR: no longer C70.1, IC21.5, VD3.C
- net N$4: no longer TP10.TP
- net NAV_I2C_SCL: no longer IC1.128, IC12.A1, R8.2
- net NAV_I2C_SDA: no longer IC1.127, IC12.A2, R13.2
- net NAV_INT0: no longer IC1.132
- net NRF_IRQ: no longer IC23.6
- net NRF_MISO: no longer IC23.5
- net NRF_MOSI: no longer IC23.4
- net NRF_SCL: no longer IC23.3
- net PWR_BUT: no longer IC1.129, VD4.C
- net PWR_OTG_MODE: no longer IC22.15, IC4.4, Q8.1, R12.2, TP83.TP
- net PWR_SHDN: no longer Q3.1, TP84.TP
- net RADIO_CE: no longer IC23.1
- net SAI_FSA: no longer IC1.111
- net SAI_MCLK: no longer IC1.115
- net SAI_SCKA: no longer IC1.113
- net SAI_SDA: no longer IC1.112
- net SAI_SDB: no longer IC1.110
- net SDR_!CAS: now also IC3.F7; no longer IC1.44, IC3.17
- net SDR_!E0: now also IC3.G9; no longer IC1.74, IC3.19
- net SDR_!RAS: now also IC3.F8; no longer IC1.46, IC3.18
- net SDR_!WE: now also IC3.F9; no longer IC1.43, IC3.16
- net SDR_BQ0: now also IC3.G7; no longer IC1.73, IC3.20
- net SDR_BQ1: now also IC3.G8; no longer IC1.75, IC3.21
- net SDR_CKE0: now also IC3.F3; no longer IC1.64, IC3.37
- net SDR_CLK: now also IC3.F2; no longer IC1.60, IC3.38
- net SDR_NBL0: now also IC3.E8; no longer IC1.42, IC3.15
- net SDR_NBL1: now also IC3.F1; no longer IC1.59, IC3.39
- net SWD_CLK: no longer SCL8.TP, X16.A11
- net SWD_IO: no longer IO.TP, X16.B3
- net SYS_LED1: no longer Q5.1
- net TS_INT: no longer IC1.7
- net TS_SCL: no longer IC1.11, R10.2, SJ3.2
- net TS_SDA: no longer IC1.10, R11.2, SJ2.2
- net UART_EXT_RX: no longer SCL10.TP, X16.A3
- net UART_EXT_TX: no longer SCL11.TP, X16.A2
- net USB_CC2: no longer TP25.TP, X16.B5
- net V_BAT: no longer IC22.20, IC22.21, R14.2
Routing:
- net 3.3V: track 792.0 -> 0.00 mm, vias 47 -> 0
- net V_INT: track 241.3 -> 0.00 mm, vias 2 -> 0
- net PWR_BUT: track 217.7 -> 0.00 mm, vias 8 -> 0
- net RINGN: track 179.3 -> 0.00 mm, vias 4 -> 0
- net 1.2V: track 168.4 -> 0.00 mm, vias 10 -> 0
- net RINGP: track 164.8 -> 0.00 mm, vias 4 -> 0
- net DMIC_DAT: track 151.1 -> 0.00 mm, vias 4 -> 0
- net DMIC_CLK: track 149.6 -> 0.00 mm, vias 4 -> 0
- net EE_I2C_SCL: track 142.1 -> 0.00 mm, vias 6 -> 0
- net EE_I2C_SDA: track 140.1 -> 0.00 mm, vias 7 -> 0
- net 2.5V: track 137.7 -> 0.00 mm, vias 7 -> 0
- net ESP_TX: track 134.3 -> 0.00 mm, vias 2 -> 0
- net ESP_RX: track 131.9 -> 0.00 mm, vias 2 -> 0
- net FMC_!OE: track 121.4 -> 0.00 mm, vias 3 -> 0
- net GPIO_FPGA1: track 116.8 -> 0.00 mm, vias 3 -> 0
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- added copper zone on layer 3, net 3.3V
Other:
- outline, holes or cut-outs redrawn
