File: redphone.sch (EAGLE design)
At the start: 241 parts, among them IC1 EP4CE15E22, IC10 74LVC1G02DCK, IC11 74LVC1G02DCK, IC12 74LVC1G02DCK, IC13 MAX1708, IC15 LSM303DLHC, IC16 EPCS4SI8N, IC17 L3GD20, IC18 WM8903, IC19 AT25SF041, IC2 STM32F429ZIT, IC20 MP34DT01, IC21 PT4181, IC22 MAX8903A, IC23 NRF24L01+, IC24 BME280, IC25 APDS-9960, IC3 MT48LC16M16A2TG, IC4 MAX8815A, IC5 TPS73025DBVT, IC6 LP3990MF-1.2, IC7 TPS63000, IC8 ESP8266, IC9 SIM800C, Q1 IRLML6402, Q10 NTA4153NT1G, Q2 NTA4153NT1G, Q4 NTA4153NT1G, Q6 IRLML6402, Q7 16MHz, Q8 NTA4153NT1G, SW1 PWR, SW2 CAM, SW3 VOL+, SW4 VOL-, X1 MICROSIM, X10 AUDIO-JACKSMD, X13 OV2640, X14 EXT, X15 DF13-4P-1.25V, X2 BAT, X3 RM68120_LCD, X7 CTS, Y1 2.4Ghz, Y3 2.4Ghz, Y4 GSM_PCB, Y5 2.4Ghz

Commit message: new modem dc-dc
Parts:
- removed C8: 100n, netcat:CAPC0402
- removed C9: 220n, netcat:CAPC0402
- removed L3: 2.2uH, netcat:LCDR
- removed R10: 1M, netcat:RESR0402
- removed R11: 220k, netcat:RESR0402
- removed R52: 12k, netcat:RESR0402
- removed R58: 100k, netcat:RESR0402
- removed TP21: 4.0v, netcat:TP06R
- removed VD2: STPS0520Z, netcat:STPS0520Z
- added L7: 2.2uH, netcat:LCDR
- added R45: 100, netcat:RESR0402
- added R46: 1M, netcat:RESR0402
- C5: value 100n -> 10u; device netcat:CAPC0402 -> netcat:CPOL-EUSMCB
- C6: value 100u -> 100n; device netcat:CPOL-EUSMCC -> netcat:CAPC0402
- IC13: value MAX1708 -> TPS63001; device netcat:MAX1708 -> netcat:TPS63000
- IC7: value TPS63000 -> TPS63001
- R51: value 27k -> 220k
Connections:
- removed net N$12: IC7.FB, R10.2, R11.1
- removed net N$15: IC13.LX, L3.P$2, VD2.A
- removed net N$98: IC13.FB, R51.1, R52.2
- new net N$10: C6.1, IC13.PS, IC13.VINA, R45.1
- new net N$28: IC13.L2, L7.P$2
- net !GSM_EN: now also IC13.EN; no longer IC13.ONA
- net 3.3V: now also IC7.FB; no longer R10.1
- net 4.0V: now also C5.+, IC13.VOUT, R46.1; no longer C5.1, C6.+, IC13.CLK, IC13.OUT, R51.2, TP21.TEST, VD2.C
- net GND: now also C5.-, C6.2, IC13.PPAD, R51.2; no longer C5.2, C6.-, C8.2, C9.2, IC13.!3.3!/5, R11.2, R52.1, R58.2
- net N$19: now also IC13.FB, R46.2, R51.1; no longer C8.1, IC13.SS/LIM, R58.1
- net N$20: now also IC13.L1, L7.P$1; no longer C9.1, IC13.REF
- net V_INT: now also IC13.VIN, R45.2; no longer IC13.!ONB, L3.P$1
Other:
- moved on the sheet: C1, C7, IC13, R51

Commit message: fix VDD_RTC on wifi chip
Connections:
- net 3.3V: no longer IC8.VDD_RTC
Changed lines of the file:
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@@
 <wire x1="-5.08" y1="-81.28" x2="-5.08" y2="-78.74" width="0.1524" layer="91"/>
 <junction x="-5.08" y="-78.74"/>
-<wire x1="-2.54" y1="-83.82" x2="-5.08" y2="-83.82" width="0.1524" layer="91"/>
-<wire x1="-5.08" y1="-83.82" x2="-5.08" y2="-81.28" width="0.1524" layer="91"/>
-<junction x="-5.08" y="-81.28"/>
 <pinref part="C15" gate="G$1" pin="1"/>
 <wire x1="-22.86" y1="-76.2" x2="-22.86" y2="-73.66" width="0.1524" layer="91"/>
@@
 <pinref part="IC8" gate="G$1" pin="VDDD"/>
 <pinref part="IC8" gate="G$1" pin="VDDPST"/>
-<pinref part="IC8" gate="G$1" pin="VDD_RTC"/>
 </segment>
 <segment>

Commit message: new pkg of wifi's crystall
Parts:
- OSC1: device netcat:CRYSTAL_SMDMINI2 -> netcat:CRYSTAL_SMDMICRO2
Changed lines of the file:
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@@
 <grid distance="0.1" unitdist="inch" unit="inch" style="lines" multiple="1" display="no" altdistance="0.01" altunitdist="inch" altunit="inch"/>
 <layers>
-<layer number="1" name="Top" color="4" fill="1" visible="yes" active="no"/>
-<layer number="2" name="Route2" color="1" fill="3" visible="yes" active="no"/>
-<layer number="3" name="Route3" color="4" fill="3" visible="yes" active="no"/>
-<layer number="4" name="Route4" color="1" fill="4" visible="yes" active="no"/>
-<layer number="5" name="Route5" color="4" fill="4" visible="yes" active="no"/>
-<layer number="6" name="Route6" color="1" fill="8" visible="yes" active="no"/>
-<layer number="7" name="Route7" color="4" fill="8" visible="yes" active="no"/>
-<layer number="8" name="Route8" color="1" fill="2" visible="yes" active="no"/>
-<layer number="9" name="Route9" color="4" fill="2" visible="yes" active="no"/>
-<layer number="10" name="Route10" color="1" fill="7" visible="yes" active="no"/>
-<layer number="11" name="Route11" color="4" fill="7" visible="yes" active="no"/>
-<layer number="12" name="Route12" color="1" fill="5" visible="yes" active="no"/>
-<layer number="13" name="Route13" color="4" fill="5" visible="yes" active="no"/>
-<layer number="14" name="Route14" color="1" fill="6" visible="yes" active="no"/>
-<layer number="15" name="Route15" color="4" fill="6" visible="yes" active="no"/>
-<layer number="16" name="Bottom" color="1" fill="1" visible="yes" active="no"/>
-<layer number="17" name="Pads" color="2" fill="1" visible="yes" active="no"/>
-<layer number="18" name="Vias" color="2" fill="1" visible="yes" active="no"/>
-<layer number="19" name="Unrouted" color="6" fill="1" visible="yes" active="no"/>
-<layer number="20" name="Dimension" color="15" fill="1" visible="yes" active="no"/>
-<layer number="21" name="tPlace" color="7" fill="1" visible="yes" active="no"/>
-<layer number="22" name="bPlace" color="7" fill="1" visible="yes" active="no"/>
-<layer number="23" name="tOrigins" color="15" fill="1" visible="yes" active="no"/>
-<layer number="24" name="bOrigins" color="15" fill="1" visible="yes" active="no"/>
-<layer number="25" name="tNames" color="7" fill="1" visible="yes" active="no"/>
-<layer number="26" name="bNames" color="7" fill="1" visible="yes" active="no"/>
-<layer number="27" name="tValues" color="7" fill="1" visible="yes" active="no"/>
-<layer number="28" name="bValues" color="7" fill="1" visible="yes" active="no"/>
+<layer number="1" name="Top" color="4" fill="1" visible="no" active="no"/>
+<layer number="2" name="Route2" color="1" fill="3" visible="no" active="no"/>
+<layer number="3" name="Route3" color="4" fill="3" visible="no" active="no"/>
+<layer number="4" name="Route4" color="1" fill="4" visible="no" active="no"/>
+<layer number="5" name="Route5" color="4" fill="4" visible="no" active="no"/>
+<layer number="6" name="Route6" color="1" fill="8" visible="no" active="no"/>
+<layer number="7" name="Route7" color="4" fill="8" visible="no" active="no"/>
+<layer number="8" name="Route8" color="1" fill="2" visible="no" active="no"/>
+<layer number="9" name="Route9" color="4" fill="2" visible="no" active="no"/>
+<layer number="10" name="Route10" color="1" fill="7" visible="no" active="no"/>
+<layer number="11" name="Route11" color="4" fill="7" visible="no" active="no"/>
+<layer number="12" name="Route12" color="1" fill="5" visible="no" active="no"/>
+<layer number="13" name="Route13" color="4" fill="5" visible="no" active="no"/>
+<layer number="14" name="Route14" color="1" fill="6" visible="no" active="no"/>
+<layer number="15" name="Route15" color="4" fill="6" visible="no" active="no"/>
+<layer number="16" name="Bottom" color="1" fill="1" visible="no" active="no"/>
+<layer number="17" name="Pads" color="2" fill="1" visible="no" active="no"/>
+<layer number="18" name="Vias" color="2" fill="1" visible="no" active="no"/>
+<layer number="19" name="Unrouted" color="6" fill="1" visible="no" active="no"/>
+<layer number="20" name="Dimension" color="15" fill="1" visible="no" active="no"/>
+<layer number="21" name="tPlace" color="7" fill="1" visible="no" active="no"/>
+<layer number="22" name="bPlace" color="7" fill="1" visible="no" active="no"/>
+<layer number="23" name="tOrigins" color="15" fill="1" visible="no" active="no"/>
+<layer number="24" name="bOrigins" color="15" fill="1" visible="no" active="no"/>
+<layer number="25" name="tNames" color="7" fill="1" visible="no" active="no"/>
+<layer number="26" name="bNames" color="7" fill="1" visible="no" active="no"/>
+<layer number="27" name="tValues" color="7" fill="1" visible="no" active="no"/>
+<layer number="28" name="bValues" color="7" fill="1" visible="no" active="no"/>
 <layer number="29" name="tStop" color="7" fill="3" visible="no" active="no"/>
 <layer number="30" name="bStop" color="7" fill="6" visible="no" active="no"/>
@@
 <layer number="35" name="tGlue" color="7" fill="4" visible="no" active="no"/>
 <layer number="36" name="bGlue" color="7" fill="5" visible="no" active="no"/>
-<layer number="37" name="tTest" color="7" fill="1" visible="yes" active="no"/>
-<layer number="38" name="bTest" color="7" fill="1" visible="yes" active="no"/>
+<layer number="37" name="tTest" color="7" fill="1" visible="no" active="no"/>
+<layer number="38" name="bTest" color="7" fill="1" visible="no" active="no"/>
 <layer number="39" name="tKeepout" color="4" fill="11" visible="no" active="no"/>
 <layer number="40" name="bKeepout" color="1" fill="11" visible="no" active="no"/>
@@
 <layer number="44" name="Drills" color="7" fill="1" visible="no" active="no"/>
 <layer number="45" name="Holes" color="7" fill="1" visible="no" active="no"/>
-<layer number="46" name="Milling" color="3" fill="1" visible="yes" active="no"/>
-<layer number="47" name="Measures" color="7" fill="1" visible="yes" active="no"/>
-<layer number="48" name="Document" color="7" fill="1" visible="yes" active="no"/>
-<layer number="49" name="Reference" color="7" fill="1" visible="yes" active="no"/>
-<layer number="50" name="dxf" color="7" fill="1" visible="yes" active="no"/>
-<layer number="51" name="tDocu" color="7" fill="1" visible="yes" active="no"/>
-<layer number="52" name="bDocu" color="7" fill="1" visible="yes" active="no"/>
-<layer number="53" name="tGND_GNDA" color="7" fill="9" visible="yes" active="no"/>
-<layer number="54" name="bGND_GNDA" color="1" fill="9" visible="yes" active="no"/>
-<layer number="56" name="wert" color="7" fill="1" visible="yes" active="no"/>
-<layer number="57" name="tCAD" color="7" fill="1" visible="yes" active="no"/>
-<layer number="59" name="tCarbon" color="7" fill="1" visible="yes" active="no"/>
-<layer number="60" name="bCarbon" color="7" fill="1" visible="yes" active="no"/>
+<layer number="46" name="Milling" color="3" fill="1" visible="no" active="no"/>
+<layer number="47" name="Measures" color="7" fill="1" visible="no" active="no"/>
+<layer number="48" name="Document" color="7" fill="1" visible="no" active="no"/>
+<layer number="49" name="Reference" color="7" fill="1" visible="no" active="no"/>
+<layer number="50" name="dxf" color="7" fill="1" visible="no" active="no"/>
+<layer number="51" name="tDocu" color="7" fill="1" visible="no" active="no"/>
+<layer number="52" name="bDocu" color="7" fill="1" visible="no" active="no"/>
+<layer number="53" name="tGND_GNDA" color="7" fill="9" visible="no" active="no"/>
+<layer number="54" name="bGND_GNDA" color="1" fill="9" visible="no" active="no"/>
+<layer number="56" name="wert" color="7" fill="1" visible="no" active="no"/>
+<layer number="57" name="tCAD" color="7" fill="1" visible="no" active="no"/>
+<layer number="59" name="tCarbon" color="7" fill="1" visible="no" active="no"/>
+<layer number="60" name="bCarbon" color="7" fill="1" visible="no" active="no"/>
 <layer number="90" name="Modules" color="5" fill="1" visible="yes" active="yes"/>
 <layer number="91" name="Nets" color="2" fill="1" visible="yes" active="yes"/>
@@
 <part name="GND44" library="netcat" deviceset="GND" device=""/>
 <part name="GND45" library="netcat" deviceset="GND" device=""/>
-<part name="OSC1" library="netcat" deviceset="CRYSTAL_SMD" device="MINI2" value="26 Mhz"/>
+<part name="OSC1" library="netcat" deviceset="CRYSTAL_SMD" device="MICRO2" value="26 Mhz"/>
 <part name="C19" library="netcat" deviceset="CAP" device="C0402" value="10p"/>
 <part name="C20" library="netcat" deviceset="CAP" device="C0402" value="10p"/>

Commit message: new 1.2/2.5 dc-dc, fix bad pinout on audiocodec
Parts:
- removed C10, C78: 100n, netcat:CAPC0402
- C7: device netcat:CPOL-EUSMCC -> netcat:CPOL-EUSMCB
- IC5: value TPS73025DBVT -> LP3990TL; device netcat:LP3985 -> netcat:LP3990TL
- IC6: value LP3990MF-1.2 -> LP3990TL; device netcat:LP3985 -> netcat:LP3990TL
Connections:
- removed net N$100: C78.1, IC6.C
- removed net N$21: C10.1, IC5.C
- net GND: no longer C10.2, C78.2

Commit message: i2c & cts tps, cap pkg fix, names fix, route fix
Parts:
- added TP21: AIN, netcat:TP06R
- added TP23: AOUT, netcat:TP06R
- added TP24: TSI, netcat:TP06R
- added TP25: MSDA, netcat:TP06R
- added TP26: MSCL, netcat:TP06R
- C1, C2, C5, C7: device netcat:CPOL-EUSMCB -> netcat:CPOL-EUSMCA
- IC1: value EP4CE15E22 -> EP4CE6E22
- IC13: value TPS63001 -> TPS63000
- IC14: value (none) -> 24LC256
Connections:
- net EE_I2C_SCL: now also TP26.TEST
- net EE_I2C_SDA: now also TP25.TEST
- net GSM_A_IN: now also TP21.TEST
- net GSM_A_OUT: now also TP23.TEST
- net TS_INT: now also TP24.TEST
Other:
- moved on the sheet: C28, C29, C3, C4, IC5, IC6, R49

Commit message: connect rtc to vbat, change mosfet type
Parts:
- removed X15: DF13-4P-1.25V, netcat:DF13-4P-1.25V
- added C8: 1u, netcat:CAPC0603
- added VD2: STPS0520Z, netcat:STPS0520Z
- Q1, Q6: value IRLML6402 -> IRLML2502
Connections:
- new net N$12: C8.1, IC2SPEC.VBAT, VD2.C
- net 3.3V: no longer IC2SPEC.VBAT, X15.2
- net FPGA_RX: no longer X15.4
- net FPGA_TX: no longer X15.3
- net GND: now also C8.2; no longer X15.1
- net V_BAT: now also VD2.A

Commit message: swap usb_cc1 to mcu_rst
Connections:
- removed net USB_CC1: IC2GPIOA.PA15, X16.CC1
- net BL_RST: now also X16.CC1
Changed lines of the file:
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@@
 <pinref part="IC2" gate="SPEC" pin="!RST"/>
+</segment>
+<segment>
+<pinref part="X16" gate="G$1" pin="CC1"/>
+<wire x1="-378.46" y1="147.32" x2="-381" y2="147.32" width="0.1524" layer="91"/>
+<label x="-378.46" y="147.32" size="1.778" layer="95"/>
 </segment>
 </net>
@@
 </segment>
 </net>
-<net name="USB_CC1" class="0">
-<segment>
-<pinref part="X16" gate="G$1" pin="CC1"/>
-<wire x1="-378.46" y1="147.32" x2="-381" y2="147.32" width="0.1524" layer="91"/>
-<label x="-378.46" y="147.32" size="1.778" layer="95"/>
-</segment>
-<segment>
-<pinref part="IC2" gate="GPIOA" pin="PA15"/>
-<wire x1="-33.02" y1="132.08" x2="-35.56" y2="132.08" width="0.1524" layer="91"/>
-<label x="-35.56" y="132.08" size="1.778" layer="95" rot="R180"/>
-</segment>
-</net>
