File: redphone.sch (EAGLE design)
At the start: 239 parts, among them IC1 EP4CE6E22, IC10 74LVC1G02DCK, IC11 74LVC1G02DCK, IC12 74LVC1G02DCK, IC13 TPS63000, IC14 24LC256, IC15 LSM303DLHC, IC16 EPCS4SI8N, IC17 L3GD20, IC18 WM8903, IC19 AT25SF041, IC2 STM32F429ZIT, IC20 MP34DT01, IC21 PT4181, IC22 MAX8903A, IC23 NRF24L01+, IC24 BME280, IC25 APDS-9960, IC3 MT48LC16M16A2TG, IC4 MAX8815A, IC5 LP3990TL, IC6 LP3990TL, IC7 TPS63001, IC8 ESP8266, IC9 SIM800C, Q1 IRLML2502, Q10 NTA4153NT1G, Q2 NTA4153NT1G, Q4 NTA4153NT1G, Q6 IRLML2502, Q7 16MHz, Q8 NTA4153NT1G, SW1 PWR, SW2 CAM, SW3 VOL+, SW4 VOL-, X1 MICROSIM, X10 AUDIO-JACKSMD, X13 OV2640, X14 EXT, X2 BAT, X3 RM68120_LCD, X7 CTS, Y1 2.4Ghz, Y3 2.4Ghz, Y4 GSM_PCB, Y5 2.4Ghz

Commit message: change fpga crystal to osc, update lbr
Parts:
- removed C53: 22p, netcat:CAPC0402
- C54: value 22p -> 100n
- OSC1: value 26 Mhz -> 26 MHz; device netcat:CRYSTAL_SMDMICRO2 -> netcat:CRYSTAL_GND2520
- OSC2, Q7: device netcat:CRYSTAL_SMDMINI2 -> netcat:CRYSTAL_GND3225
- OSC3: device netcat:CRYSTALMICRO32 -> netcat:CRYSTAL3215
- OSC4: value 48 mhz -> 48 MHz; device netcat:CRYSTAL_SMDMINI2 -> netcat:OSC3225
Connections:
- removed net OSCO1: C54.2, IC1CLK.IO_25/CLK3, OSC4.1
- net 3.3V: now also C54.1, OSC4.VCC
- net GND: now also C54.2; no longer C53.1, C54.1
- net OSCI1: now also OSC4.OUT; no longer C53.2, OSC4.2
Other:
- moved on the sheet: C54

Commit message: lowdrop en ctrl from stm
Parts:
- removed SCL1: PB12, netcat:TP06R
- VD2: value STPS0520Z -> BAS516; device netcat:STPS0520Z -> netcat:DIODE
Connections:
- removed net N$95: IC2GPIOB.PB12, SCL1.TEST
- new net FPGA_EN: IC2GPIOB.PB12, IC5.EN, IC6.EN
- net V_INT: no longer IC5.EN, IC6.EN
Other:
- moved on the sheet: C30, C31, C8, IC2PWR

Commit message: added ds18b20, udfn pack for eeprom, some route fix
Parts:
- removed TP13: TSCL, netcat:TP06R
- removed TP25: MSDA, netcat:TP06R
- removed TP26: MSCL, netcat:TP06R
- removed TP5: TSDA, netcat:TP06R
- added IC26: DS18B20U, netcat:DS18B20U
- added R10, R11: 4.7k, netcat:RESR0402
- added SJ2, SJ3: (no value), netcat:SJ2
- IC14: device netcat:24LC256-I/SN -> netcat:AT24C64D
- OSC2: value 8 mhz -> 8 MHz
- OSC3: value 32.768k -> 32.768 KHz
- R13, R38, R39, R8: value 10k -> 4.7k
- R15: value 1M -> 300k
Connections:
- new net 1W: IC1CLK.IO_23/CLK1, IC26.1W
- net 3.3V: now also IC26.VCC, R10.1, R11.1
- net EE_I2C_SCL: now also SJ3.1; no longer TP26.TEST
- net EE_I2C_SDA: now also SJ2.1; no longer TP25.TEST
- net GND: now also IC26.GND
- net TS_SCL: now also R10.2, SJ3.2; no longer TP13.TEST
- net TS_SDA: now also R11.2, SJ2.2; no longer TP5.TEST
Other:
- moved on the sheet: R38, R39

Commit message: new battery connection mechanism
Parts:
- removed X2: BAT, netcat:M03
- U$3: value GALAXY_S3MINI_BATTARY -> GALAXY_BATTARY_S4; device netcat:GALAXY_S3MINI_BATTARY -> netcat:GALAXY_BATTARY_S4
Connections:
- net GND: no longer X2.3
- net V_BAT: no longer X2.1
Changed lines of the file:
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@@
 <part name="IC11" library="netcat" deviceset="74LVC1G02" device="DCK" value="74LVC1G02DCK"/>
 <part name="X3" library="netcat" deviceset="RM68120_LCD" device=""/>
-<part name="GND13" library="netcat" deviceset="GND" device=""/>
 <part name="Q6" library="netcat" deviceset="MOSFET_P" device="" value="IRLML2502"/>
 <part name="R9" library="netcat" deviceset="RES" device="R0402" value="100"/>
@@
 <part name="GND78" library="netcat" deviceset="GND" device=""/>
 <part name="C71" library="netcat" deviceset="CAP" device="C0402" value="100n"/>
-<part name="X2" library="netcat" deviceset="M03" device="" value="BAT"/>
 <part name="C72" library="netcat" deviceset="CAP" device="C0402" value="100n"/>
 <part name="GND79" library="netcat" deviceset="GND" device=""/>
@@
 <part name="2.5V6" library="netcat" deviceset="2.5V" device=""/>
 <part name="GND87" library="netcat" deviceset="GND" device=""/>
-<part name="U$3" library="netcat" deviceset="GALAXY_S3MINI_BATTARY" device=""/>
+<part name="U$3" library="netcat" deviceset="GALAXY_BATTARY" device="_S4"/>
 <part name="C73" library="netcat" deviceset="CAP" device="C0402" value="100n"/>
 <part name="IC24" library="netcat" deviceset="BME280" device=""/>
@@
 <instance part="IC11" gate="A" x="-304.8" y="27.94"/>
 <instance part="X3" gate="G$1" x="218.44" y="-35.56"/>
-<instance part="GND13" gate="GND" x="-274.32" y="99.06" rot="MR0"/>
 <instance part="Q6" gate="G$1" x="-251.46" y="154.94" smashed="yes" rot="MR90">
 <attribute name="NAME" x="-261.62" y="165.1" size="1.778" layer="95" rot="MR180"/>
@@
 <instance part="GND78" gate="GND" x="-447.04" y="-88.9"/>
 <instance part="C71" gate="G$1" x="444.5" y="-63.5"/>
-<instance part="X2" gate="G$1" x="-271.78" y="109.22"/>
 <instance part="C72" gate="G$1" x="-302.26" y="88.9" rot="R180"/>
 <instance part="GND79" gate="GND" x="-302.26" y="81.28"/>
@@
 </segment>
 <segment>
-<pinref part="X2" gate="G$1" pin="3"/>
-<pinref part="GND13" gate="GND" pin="GND"/>
-<wire x1="-271.78" y1="104.14" x2="-274.32" y2="104.14" width="0.1524" layer="91"/>
-<wire x1="-274.32" y1="104.14" x2="-274.32" y2="101.6" width="0.1524" layer="91"/>
-</segment>
-<segment>
 <pinref part="X6" gate="G$1" pin="1"/>
 <pinref part="GND80" gate="GND" pin="GND"/>
@@
 <net name="V_BAT" class="0">
 <segment>
-<wire x1="-281.94" y1="109.22" x2="-274.32" y2="109.22" width="0.1524" layer="91"/>
-<wire x1="-274.32" y1="109.22" x2="-271.78" y2="109.22" width="0.1524" layer="91"/>
-<junction x="-274.32" y="109.22"/>
-<label x="-274.32" y="111.76" size="1.778" layer="95" rot="MR0"/>
-<wire x1="-274.32" y1="109.22" x2="-274.32" y2="111.76" width="0.1524" layer="91"/>
+<wire x1="-281.94" y1="109.22" x2="-279.4" y2="109.22" width="0.1524" layer="91"/>
+<label x="-279.4" y="109.22" size="1.778" layer="95" rot="MR180"/>
 <pinref part="R14" gate="G$1" pin="2"/>
 <wire x1="-281.94" y1="104.14" x2="-281.94" y2="109.22" width="0.1524" layer="91"/>
@@
 <wire x1="-281.94" y1="109.22" x2="-317.5" y2="109.22" width="0.1524" layer="91"/>
 <pinref part="IC22" gate="G$1" pin="BAT"/>
-<pinref part="X2" gate="G$1" pin="1"/>
 </segment>
 <segment>

Commit message: added gps, combine sim and sd slots in one
Parts:
- removed X5: (no value), netcat:MICRO_SD
- added C10: (no value), netcat:CAPC0402
- added C9: 100p, netcat:CAPC0402
- added IC27: MC-1010-G, netcat:MC-1010-G
- added IC28: MAX2659, netcat:MAX2659
- added L3: (no value), netcat:L0402
- added Y2: (no value), netcat:ANTENNA_CHIP2X9
- X1: value MICROSIM -> MOLEX_SIM_SD; device netcat:MICROSIM -> netcat:MOLEX_SIM_SD
Connections:
- new net GPS_RX: IC27.RX, IC2GPIOF.PF7
- new net GPS_TX: IC27.TX, IC2GPIOF.PF6
- new net N$21: C10.1, Y2.FEED
- new net N$61: C10.2, L3.P$1
- new net N$72: IC28.RF_IN, L3.P$2
- new net RF_OUT: IC27.RF_IN, IC28.RF_OUT
- new net VCC_RF: C9.1, IC27.VCC_RF, IC28.!SHDN, IC28.VCC
- net 3.3V: now also IC27.VCC, IC27.V_BCKP, X1G$1.VCC, X1SD.VCC; no longer X1.VCC, X5.VCC
- net GND: now also C9.2, IC27.GND, IC28.GND, X1SD.GND; no longer X1.GND, X5.GND
- net SDHC_ST: now also X1SD.ST; no longer X5.ST
- net SDIO0: now also X1SD.DAT0/MISO; no longer X5.MISO/DAT0
- net SDIO1: now also X1SD.DAT1; no longer X5.DAT1
- net SDIO2: now also X1SD.DAT2; no longer X5.DAT2
- net SDIO3: now also X1SD.DAT3/CS; no longer X5.CS/DAT3
- net SDIO_CLK: now also X1SD.CLK; no longer X5.CLK
- net SDIO_CMD: now also X1SD.CMD/MOSI; no longer X5.MOSI/CMD
- net SIM_CLK: now also X1G$1.CLK; no longer X1.CLK
- net SIM_DATA: now also X1G$1.I/O; no longer X1.I/O
- net SIM_DET: no longer X1.ID
- net SIM_RST: now also X1G$1.RST; no longer X1.RST
- net SIM_VDD: now also X1G$1.VPP; no longer X1.VPP

Commit message: upd route, new pwr logic
Parts:
- removed C26: 1.0p, netcat:CAPC0402
- removed IC10, IC11, IC12: 74LVC1G02DCK, netcat:74LVC1G02DCK
- removed R6, R7: 100k, netcat:RESR0402
- removed TP20: VSYS, netcat:TP06R
- removed TP22: SHDN, netcat:TP06R
- added Q3: BCR133W, netcat:NPNSOT323
- added VD4: (no value), netcat:DIODE
Connections:
- removed net !BAT_EN: IC10.B, IC11.Y
- removed net BAT_EN: IC10.Y, IC11.A, Q1.G, R7.1
- removed net N$7: IC10.A, IC12.Y
- new net N$15: Q1.G, Q3.C, R4.1, VD4.C
- net 3.3V: now also X1SIM.VCC; no longer X1G$1.VCC
- net ANT: no longer C26.2
- net GND: now also Q3.E; no longer C26.1, IC10.GND, IC11.GND, IC12.GND, R4.1
- net PWR_BUT: now also VD4.A; no longer IC12.A, IC12.B, R6.1
- net PWR_SHDN: now also Q3.B; no longer IC11.B, R4.2, TP22.TEST
- net SIM_CLK: now also X1SIM.CLK; no longer X1G$1.CLK
- net SIM_DATA: now also X1SIM.I/O; no longer X1G$1.I/O
- net SIM_RST: now also X1SIM.RST; no longer X1G$1.RST
- net SIM_VDD: now also X1SIM.VPP; no longer X1G$1.VPP
- net V_SYS: now also R4.2; no longer IC10.VCC, IC11.VCC, IC12.VCC, R6.2, R7.2, TP20.TEST
Other:
- moved on the sheet: R4

Commit message: upd route, fix mdl connectors
Parts:
- removed R9: 100, netcat:RESR0402
- added TP5: IO88, netcat:TP06R
- added X2: (no value), netcat:PLS2-1X01
- X14: value EXT -> UFL
Connections:
- net MDL0 renamed FPGA_IO0
- net MDL1 renamed FPGA_IO1
- new net FPGA_IO2: IC1CLK.IO_90/CLK5, X4.1
- new net FPGA_IO3: IC1CLK.IO_91/CLK4, X6.1
- new net N$7: IC1CLK.IO_88/CLK7, TP5.TEST
- net 3.3V: now also X2.1; no longer X4.1
- net GND: no longer X6.1
- net N$9: no longer R9.1
- net V_INT: no longer R9.2
Other:
- moved on the sheet: C54, OSC4, X12, X6

Commit message: touch keyboard backlight, changed BAT_SENS input
Parts:
- removed R50: 330, netcat:RESR0402
- added LED7: (no value), netcat:LEDLED0603
- added Q5: NTA4153NT1G, netcat:MOSFET_NSOT-416
Connections:
- removed net N$96: LED6.A, R50.1
- new net N$73: LED6.C, LED7.C, Q5.D
- net 3.3V: now also LED6.A, LED7.A
- net BAT_SENS: now also IC2GPIOF.PF8; no longer IC2GPIOB.PB1
- net GND: now also Q5.S; no longer LED6.C
- net SYS_LED1: now also Q5.G; no longer R50.2
Other:
- moved on the sheet: IC27, LED6, R28, SW2, SW4
