File: redphone.sch (EAGLE design)
At the start: 227 parts, among them IC1 EP4CE22U14I7N, IC10 MPU9250, IC11 PCA9633TK, IC12 BME280, IC13 W25Q64FV, IC14 MC-1010-G, IC15 MAX2659, IC2 STM32F429NI, IC20 MP34DT01, IC25 APDS-9960, IC3 MT48LC16M16A2B4, IC4 MT48LC16M16A2B4, IC5 W25Q64FV, IC6 SIM800H, IC7 TPS65217, IC8 ESP8266, IC9 WM8903, M1 VIBRO, Q1 IRLML2502, Q2 IRLML2502, Q3 IRLML2502, SW1 PWR, SW3 VOL+, SW4 VOL-, X1 USB, X2 OV5647, X3 RM68120_LCD, X4 MICRO_SIM_SDS8, X5 LG_P715_TS, X7 AUDIO-JACKSMD, X8 FPC_I9500_BAT_CON, Y1 2.4Ghz, Y3 2.4Ghz, Y4 GSM_PCB

Commit message: fix DCDC2 res
Parts:
- L4: value 2.2uH -> 18uH
Connections:
- removed net N$16: IC7.VDCDC2, R34.1
- new net N$18: IC7.VDCDC2, R31.1, R34.1
- net 4.0V: no longer R31.1
Other:
- moved on the sheet: R31, R34
Changed lines of the file:
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@@
 <part name="L2" library="netcat" deviceset="L" device="-2520" value="2.2uH"/>
 <part name="L3" library="netcat" deviceset="L" device="-2520" value="2.2uH"/>
-<part name="L4" library="netcat" deviceset="L" device="-2520" value="2.2uH"/>
+<part name="L4" library="netcat" deviceset="L" device="-2520" value="18uH"/>
 <part name="C3" library="netcat" deviceset="CAP" device="0603" value="0.1u, 6.3v"/>
 <part name="C4" library="netcat" deviceset="CAP" device="1206" value="10u, 10v"/>
@@
 <attribute name="VALUE" x="127" y="-71.12" size="1.27" layer="96" align="top-center"/>
 </instance>
-<instance part="R31" gate="G$1" x="114.3" y="-10.16" smashed="yes">
-<attribute name="NAME" x="110.49" y="-8.6614" size="1.778" layer="95"/>
-<attribute name="VALUE" x="110.49" y="-13.462" size="1.778" layer="96"/>
-</instance>
-<instance part="R34" gate="G$1" x="93.98" y="-5.08" smashed="yes">
-<attribute name="NAME" x="90.17" y="-3.5814" size="1.778" layer="95"/>
-<attribute name="VALUE" x="90.17" y="-8.382" size="1.778" layer="96"/>
+<instance part="R31" gate="G$1" x="119.38" y="-10.16" smashed="yes">
+<attribute name="NAME" x="115.57" y="-8.6614" size="1.778" layer="95"/>
+<attribute name="VALUE" x="115.57" y="-13.462" size="1.778" layer="96"/>
+</instance>
+<instance part="R34" gate="G$1" x="99.06" y="-5.08" smashed="yes">
+<attribute name="NAME" x="95.25" y="-3.5814" size="1.778" layer="95"/>
+<attribute name="VALUE" x="95.25" y="-8.382" size="1.778" layer="96"/>
 </instance>
 <instance part="R35" gate="G$1" x="0" y="30.48" smashed="yes" rot="R90">
@@
 <pinref part="R31" gate="G$1" pin="2"/>
 <wire x1="162.56" y1="-17.78" x2="162.56" y2="-20.32" width="0.1524" layer="91"/>
-<wire x1="119.38" y1="-10.16" x2="154.94" y2="-10.16" width="0.1524" layer="91"/>
+<wire x1="124.46" y1="-10.16" x2="154.94" y2="-10.16" width="0.1524" layer="91"/>
 <wire x1="154.94" y1="-10.16" x2="154.94" y2="-17.78" width="0.1524" layer="91"/>
 <wire x1="154.94" y1="-17.78" x2="162.56" y2="-17.78" width="0.1524" layer="91"/>
@@
 <pinref part="U$2" gate="G$1" pin="4.0V"/>
 <pinref part="L2" gate="G$1" pin="P$2"/>
-<wire x1="104.14" y1="-5.08" x2="162.56" y2="-5.08" width="0.1524" layer="91"/>
+<wire x1="109.22" y1="-5.08" x2="162.56" y2="-5.08" width="0.1524" layer="91"/>
 <wire x1="162.56" y1="-5.08" x2="167.64" y2="-5.08" width="0.1524" layer="91"/>
-<wire x1="81.28" y1="0" x2="104.14" y2="0" width="0.1524" layer="91"/>
-<wire x1="104.14" y1="0" x2="104.14" y2="-5.08" width="0.1524" layer="91"/>
+<wire x1="81.28" y1="0" x2="109.22" y2="0" width="0.1524" layer="91"/>
+<wire x1="109.22" y1="0" x2="109.22" y2="-5.08" width="0.1524" layer="91"/>
 <pinref part="C10" gate="G$1" pin="+"/>
 <wire x1="162.56" y1="-7.62" x2="162.56" y2="-5.08" width="0.1524" layer="91"/>
 <junction x="162.56" y="-5.08"/>
 <pinref part="R34" gate="G$1" pin="2"/>
-<wire x1="99.06" y1="-5.08" x2="104.14" y2="-5.08" width="0.1524" layer="91"/>
-<junction x="104.14" y="-5.08"/>
-<pinref part="R31" gate="G$1" pin="1"/>
-<wire x1="109.22" y1="-10.16" x2="104.14" y2="-10.16" width="0.1524" layer="91"/>
-<wire x1="104.14" y1="-10.16" x2="104.14" y2="-5.08" width="0.1524" layer="91"/>
+<wire x1="104.14" y1="-5.08" x2="109.22" y2="-5.08" width="0.1524" layer="91"/>
+<junction x="109.22" y="-5.08"/>
 </segment>
 </net>
@@
 </segment>
 </net>
-<net name="N$16" class="0">
-<segment>
+<net name="N$18" class="0">
+<segment>
+<pinref part="R31" gate="G$1" pin="1"/>
+<wire x1="114.3" y1="-10.16" x2="88.9" y2="-10.16" width="0.1524" layer="91"/>
 <pinref part="IC7" gate="G$1" pin="VDCDC2"/>
 <pinref part="R34" gate="G$1" pin="1"/>
 <wire x1="68.58" y1="-5.08" x2="88.9" y2="-5.08" width="0.1524" layer="91"/>
-</segment>
-</net>
+<wire x1="88.9" y1="-5.08" x2="93.98" y2="-5.08" width="0.1524" layer="91"/>
+<wire x1="88.9" y1="-10.16" x2="88.9" y2="-5.08" width="0.1524" layer="91"/>
+<junction x="88.9" y="-5.08"/>
+</segment>
+</net>

Commit message: added ISET1 res, USB pwr input is AC now
Parts:
- added R36: 10k, netcat:RESR0402
Connections:
- new net N$16: IC7.ISET1, R36.2
- net GND: now also R36.1
- net V_USB: now also IC7.AC; no longer IC7.USB
Other:
- moved on the sheet: C5, Q1, R8, X1

Commit message: updeted LCD connector, connected 35 pin to GND
Connections:
- net LCD_WR: now also X3.WR/SCL; no longer X3.WR
Other:
- moved on the sheet: R48, X3

Commit message: remove bat & bat connector, update chip ant silk, added led for modem status
Parts:
- removed BATTARY_PLACE: GALAXY_BATTARY_S4, netcat:GALAXY_BATTARY_S4
- removed TP3, TP4, TP5, TP6: (no value), netcat:TP_HOLE
- removed X8: FPC_I9500_BAT_CON, netcat:FPC_I9500_BAT_CON
- added LOGO3: REDPHONE_LABLE, netcat:REDPHONE_LABLE
- added R37: 1k, netcat:RESR0402
- added VD7: G, netcat:LED0603
Connections:
- removed net GND_BAT2: TP3.P$1, TP4.P$1, TP6.P$1
- new net GSM_ST: IC6.STATUS, R37.2
- new net N$19: R37.1, VD7.A
- net GND: now also VD7.C
- net GND_BAT: no longer X8.GND
- net V_BAT2: no longer X8.VBAT
Other:
- moved on the sheet: Q2, Q3, R14, R15, R25, R44, SW3, SW4, TP10, TP11, TP12, TP13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

Commit message: pwr refactoring, auto pwr disable for sim-sd
Parts:
- removed C65, C75: 4.7u, netcat:CPOL-EUSMCA
- removed R16: 2om, netcat:RESR0805
- removed R25: 100k, netcat:RESR0402
- added Q4: IRLML2502, netcat:MOSFET_PSOT23
- added R38: 10k, netcat:RESR0402
- C11, C12, C13, C16, C5, C53, C6, C68, C7, C9: device netcat:CPOL-EUSMCA -> netcat:CAP0805
- C4: device netcat:CAP1206 -> netcat:CAP0805
Connections:
- removed net VCC_DIRTY: C75.+, R16.1, TP11.P$1
- new net N$22: Q4.D, X4SD.VCC, X4SIM.VCC
- net 1.2V: now also C7.1; no longer C7.+
- net 2.5V: now also C6.1; no longer C6.+
- net 3.3V: now also C11.1, Q4.S, R38.1, TP11.P$1; no longer C11.+, C65.+, R16.2, R25.1, X4SD.VCC, X4SIM.VCC
- net 4.0V: now also C68.1; no longer C68.+
- net GND: now also C11.2, C12.2, C13.2, C16.2, C5.2, C53.2, C6.2, C68.2, C7.2, C9.2; no longer C11.-, C12.-, C13.-, C16.-, C5.-, C53.-, C6.-, C65.-, C68.-, C7.-, C75.-, C9.-
- net SDHC_ST: now also Q4.G, R38.2; no longer R25.2
- net V_BAT: now also C9.1; no longer C9.+
- net V_MCU: now also C12.1; no longer C12.+
- net V_SENS: now also C13.1; no longer C13.+
- net V_SND: now also C16.1; no longer C16.+
- net V_SYS: now also C53.1; no longer C53.+
- net V_USB: now also C5.1; no longer C5.+

Commit message: now used new type of buttons
Parts:
- removed SW1: PWR, netcat:SW_GND
- added SW2: (no value), netcat:SW-YD
- SW3: value VOL+ -> (none); device netcat:SW_GND -> netcat:SW-YD
- SW4: value VOL- -> (none); device netcat:SW_GND -> netcat:SW-YD
- renumbered IC20 to IC16, IC25 to IC17
Connections:
- net GND: now also SW2.1; no longer SW1.1, SW1.GND, SW3.GND, SW4.GND
- net PWR_PB: now also SW2.2; no longer SW1.2

Commit message: added some testpoints
Parts:
- added TP3: TX, netcat:TP10R
- added TP4: RX, netcat:TP10R
- added TP_CLK: CLK, netcat:TP10R
- added TP_DI: DI, netcat:TP10R
- added TP_PJ1: PJ1, netcat:TP10R
- renumbered TP25 to TP_PJ0
Connections:
- new net N$23: IC2J.PJ1, TP_PJ1.TEST
- net EPCS_ASDI: now also TP_DI.TEST
- net EPCS_DCLK: now also TP_CLK.TEST
- net USB_CC1: now also TP3.TEST
- net USB_CC2: now also TP4.TEST

Commit message: esp8266 was replaced by esp32
Parts:
- removed IC8: ESP8266, netcat:ESP8266
- removed R17, R18, R42: 100k, netcat:RESR0402
- removed R20: 12k, netcat:RESR0402
- added C65: 10nF, netcat:CAP0402
- added C75: 3n, netcat:CAP0402
- added IC18: (no value), netcat:ESP32
- added R16: 20k, netcat:RESR0402
- added TP_ESP_TCK: TCK, netcat:TP10R
- added TP_ESP_TDI: TDI, netcat:TP10R
- added TP_ESP_TDO: TDO, netcat:TP10R
- added TP_TMS: TMS, netcat:TP10R
Connections:
- removed net GPIO15: IC8.MTDO/SPICS/GPIO15, R23.2
- removed net N$103: IC8.GPIO5, R21.1
- removed net N$47: IC8.LNA, L6.P$1
- removed net N$71: IC8.SPICS2/GPIO0, R42.2
- removed net N$92: IC8.!EXT_RSTB, R18.1
- removed net N$94: IC8.GPIO2, R17.2
- new net N$25: IC18.LNA_IN, L6.P$1
- new net N$28: IC18.GPIO15/TDO, R23.2, TP_ESP_TDO.TEST
- new net N$30: C75.2, IC18.CAP2, R16.2
- new net N$31: IC18.GPIO14/TMS, TP_TMS.TEST
- new net N$32: IC18.GPIO12/TDI, TP_ESP_TDI.TEST
- new net N$33: IC18.GPIO13/TCK, TP_ESP_TCK.TEST
- new net N$34: IC18.GPIO5, R21.1
- net 3.3V: now also IC18.VDD3P3, IC18.VDD3P3_CPU, IC18.VDD3P3_RTC, IC18.VDDA, IC18.VDD_SDIO; no longer IC8.VDD3P3, IC8.VDDA, IC8.VDDD, IC8.VDDPST, R17.1, R18.2, R42.1
- net ESP_CE: now also IC18.CE; no longer IC8.CHIP_EN
- net ESP_RX: now also IC18.GPIO3/U0RXD; no longer IC8.U0RXD
- net ESP_TX: now also IC18.GPIO1/U0TXD; no longer IC8.U0TXD
- net GND: now also C65.2, IC18.GND; no longer IC8.GND, R20.1
- net N$24: now also C65.1, C75.1, IC18.CAP1, R16.1; no longer IC8.RES12K, R20.2
- net N$26: now also IC18.XTALN; no longer IC8.XTAL_OUT
- net N$27: now also IC18.XTALP; no longer IC8.XTAL_IN
- net SD_!HD!: now also IC18.GPIO9/SPIHD; no longer IC8.SPIHD/SD_DATA_2
- net SD_!WP!: now also IC18.GPIO10/SPIWP; no longer IC8.SPIWP/SD_DATA_3
- net SD_CLK: now also IC18.GPIO6/SPICLK; no longer IC8.SPICLK/SD_CLK
- net SD_CS0: now also IC18.GPIO11/SPICS0; no longer IC8.SPICS0/SD_CMD
- net SD_SI: now also IC18.GPIO8/SPID; no longer IC8.SPID/SD_DATA_1
- net SD_SO: now also IC18.GPIO7/SPIQ; no longer IC8.SPIQ/SD_DATA_0
Other:
- moved on the sheet: C14, C15, C19, C20, C67, L5, L6, QZ3, R21, R23, Y1
